File: pcb/espander_100x_i2c/espander_100x_i2c.kicad_sch (KiCad schematic)
At the start: 5 parts, among them J1 DG127A-5.08-06P-14-00AH, J2 DG127A-5.08-06P-14-00AH, J3 DG127A-5.08-06P-14-00AH, J4 DG127A-5.08-06P-14-00AH, U1 MCP23017_SP

Commit message: Refactor code structure for improved readability and maintainability
Other:
- sheet U3 renamed U3 - U4
- added sheet U5 (U5.kicad_sch)
- added sheet U6 (U6.kicad_sch)
- added sheet U7 - U8 (U7.kicad_sch)
Changed lines of the file:
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@@
 		)
 	)
-	(global_label "U2-GPB7"
-		(shape output)
-		(at 24.13 191.77 0)
+	(global_label "U3-GPB5"
+		(shape bidirectional)
+		(at 43.18 166.37 0)
 		(fields_autoplaced yes)
 		(effects
@@
 		)
 		(property "Intersheetrefs" "${INTERSHEET_REFS}"
-			(at 36.2471 191.77 0)
+			(at 56.4084 166.37 0)
 			(effects
 				(font
@@
 		)
 	)
-	(global_label "SDA"
+	(global_label "U3-GPB6"
 		(shape bidirectional)
-		(at 35.56 184.15 180)
+		(at 55.88 162.56 180)
 		(fields_autoplaced yes)
 		(effects
@@
 		)
 		(property "Intersheetrefs" "${INTERSHEET_REFS}"
-			(at 27.8954 184.15 0)
+			(at 42.6516 162.56 0)
 			(effects
 				(font
@@
 		)
 	)
-	(global_label "SCK"
-		(shape bidirectional)
-		(at 35.56 180.34 180)
+	(global_label "U2-GPB7"
+		(shape output)
+		(at 24.13 170.18 0)
 		(fields_autoplaced yes)
 		(effects
@@
 				(size 1.27 1.27)
 			)
+			(justify left)
+		)
+		(property "Intersheetrefs" "${INTERSHEET_REFS}"
+			(at 36.2471 170.18 0)
+			(effects
+				(font
+					(size 1.27 1.27)
+				)
+				(justify left)
+				(hide yes)
+			)
+		)
+	)
+	(global_label "U3-GPB7"
+		(shape output)
+		(at 44.45 170.18 0)
+		(fields_autoplaced yes)
+		(effects
+			(font
+				(size 1.27 1.27)
+			)
+			(justify left)
+		)
+		(property "Intersheetrefs" "${INTERSHEET_REFS}"
+			(at 56.5671 170.18 0)
+			(effects
+				(font
+					(size 1.27 1.27)
+				)
+				(justify left)
+				(hide yes)
+			)
+		)
+	)
+	(global_label "SDA"
+		(shape bidirectional)
+		(at 35.56 162.56 180)
+		(fields_autoplaced yes)
+		(effects
+			(font
+				(size 1.27 1.27)
+			)
 			(justify right)
 		)
 		(property "Intersheetrefs" "${INTERSHEET_REFS}"
-			(at 27.714 180.34 0)
+			(at 27.8954 162.56 0)
+			(effects
+				(font
+					(size 1.27 1.27)
+				)
+				(justify right)
+				(hide yes)
+			)
+		)
+	)
+	(global_label "SCK"
+		(shape bidirectional)
+		(at 35.56 158.75 180)
+		(fields_autoplaced yes)
+		(effects
+			(font
+				(size 1.27 1.27)
+			)
+			(justify right)
+		)
+		(property "Intersheetrefs" "${INTERSHEET_REFS}"
+			(at 27.714 158.75 0)
 			(effects
 				(font
@@
 		)
 	)
-	(global_label "U2-GPB6"
+	(global_label "U3-GPB4"
 		(shape bidirectional)
-		(at 22.86 187.96 0)
+		(at 55.88 158.75 180)
 		(fields_autoplaced yes)
 		(effects
@@
 				(size 1.27 1.27)
 			)
+			(justify right)
+		)
+		(property "Intersheetrefs" "${INTERSHEET_REFS}"
+			(at 42.6516 158.75 0)
+			(effects
+				(font
+					(size 1.27 1.27)
+				)
+				(justify right)
+				(hide yes)
+			)
+		)
+	)
+	(global_label "U2-GPB6"
+		(shape bidirectional)
+		(at 22.86 166.37 0)
+		(fields_autoplaced yes)
+		(effects
+			(font
+				(size 1.27 1.27)
+			)
 			(justify left)
 		)
 		(property "Intersheetrefs" "${INTERSHEET_REFS}"
-			(at 36.0884 187.96 0)
+			(at 36.0884 166.37 0)
 			(effects
 				(font
@@
 	)
 	(sheet
-		(at 18.034 178.308)
-		(size 18.288 16.256)
+		(at 18.034 156.21)
+		(size 18.288 38.354)
 		(exclude_from_sim no)
 		(in_bom yes)
@@
 		)
 		(property "Sheetname" "U2"
-			(at 18.034 177.5964 0)
+			(at 18.034 155.4984 0)
 			(effects
 				(font
@@
 	)
 	(sheet
-		(at 39.6494 178.5366)
-		(size 17.2466 16.1798)
+		(at 60.96 156.21)
+		(size 17.2466 38.5064)
 		(exclude_from_sim no)
 		(in_bom yes)
@@
 			(color 0 0 0 0.0000)
 		)
-		(property "Sheetname" "U3"
-			(at 39.6494 177.825 0)
-			(effects
-				(font
+		(property "Sheetname" "U5"
+			(at 60.96 155.4984 0)
+			(effects
+				(font
+					(size 1.27 1.27)
+				)
+				(justify left bottom)
+			)
+		)
+		(property "Sheetfile" "U5.kicad_sch"
+			(at 60.96 195.301 0)
+			(effects
+				(font
+					(size 1.27 1.27)
+				)
+				(justify left top)
+			)
+		)
+		(instances
+			(project "espander_100x_i2c"
+				(path "/824ceec5-564f-405b-8bea-e5a9f7aa2926"
+					(page "4")
+				)
+			)
+		)
+	)
+	(sheet
+		(at 82.55 156.21)
+		(size 17.2466 38.5064)
+		(exclude_from_sim no)
+		(in_bom yes)
+		(on_board yes)
+		(dnp no)
+		(fields_autoplaced yes)
+		(stroke
+			(width 0.1524)
+			(type solid)
+		)
+		(fill
+			(color 0 0 0 0.0000)
+		)
+		(property "Sheetname" "U6"
+			(at 82.55 155.4984 0)
+			(effects
+				(font
+					(size 1.27 1.27)
+				)
+				(justify left bottom)
+			)
+		)
+		(property "Sheetfile" "U6.kicad_sch"
+			(at 82.55 195.301 0)
+			(effects
+				(font
+					(size 1.27 1.27)
+				)
+				(justify left top)
+			)
+		)
+		(instances
+			(project "espander_100x_i2c"
+				(path "/824ceec5-564f-405b-8bea-e5a9f7aa2926"
+					(page "5")
+				)
+			)
+		)
+	)
+	(sheet
+		(at 104.14 156.21)
+		(size 17.2466 38.5064)
+		(exclude_from_sim no)
+		(in_bom yes)
+		(on_board yes)
+		(dnp no)
+		(fields_autoplaced yes)
+		(stroke
+			(width 0.1524)
+			(type solid)
+		)
+		(fill
+			(color 0 0 0 0.0000)
+		)
+		(property "Sheetname" "U7 - U8"
+			(at 104.14 155.4984 0)
+			(effects
+				(font
+					(size 1.27 1.27)
+				)
+				(justify left bottom)
+			)
+		)
+		(property "Sheetfile" "U7.kicad_sch"
+			(at 104.14 195.301 0)
+			(effects
+				(font
+					(size 1.27 1.27)
+				)
+				(justify left top)
+			)
+		)
+		(instances
+			(project "espander_100x_i2c"
+				(path "/824ceec5-564f-405b-8bea-e5a9f7aa2926"
+					(page "6")
+				)
+			)
+		)
+	)
+	(sheet
+		(at 39.6494 156.21)
+		(size 17.2466 38.5064)
+		(exclude_from_sim no)
+		(in_bom yes)
+		(on_board yes)
+		(dnp no)
+		(fields_autoplaced yes)
+		(stroke
+			(width 0.1524)
+			(type solid)
+		)
+		(fill
+			(color 0 0 0 0.0000)
+		)
+		(property "Sheetname" "U3 - U4"
+			(at 39.6494 155.4984 0)
+			(effects
+				(font

Commit message: Resync
Other:
- added sheet esp32 (esp32.kicad_sch)
- moved on the sheet: J1, J2, J3, J4, U1

Commit message: resync
Parts:
- added C1, C2: 100nF, Capacitor_THT:C_Disc_D3.0mm_W2.0mm_P2.50mm, symbol Device:C_Polarized
- added U10, U12: ITS716G, Package_SO:SOIC-20W_7.5x12.8mm_P1.27mm, symbol Driver_FET:ITS716G
- added U11, U9: LTV-847, Package_DIP:DIP-16_W7.62mm, symbol Isolator:LTV-847
Connections:
- net GND: now also C1.2, C2.2, U10.2 (GND1/2), U10.6 (GND3/4), U11.11, U11.13, U11.15, U11.2, U11.4, U11.6, U11.8, U11.9, U12.2 (GND1/2), U12.6 (GND3/4), U9.11, U9.13, U9.15, U9.2, U9.4, U9.6, U9.8, U9.9
- net U1-GPA0: now also U11.16; no longer J4.3
- net U1-GPA1: now also U11.14; no longer J4.4
- net U1-GPA2: now also U11.12; no longer J4.5
- net U1-GPA3: now also U11.10; no longer J4.6
- net U1-GPA4: now also U12.9 (IN4); no longer J3.4
- net U1-GPA5: now also U12.7 (IN3); no longer J3.3
- net U1-GPA6: now also U12.5 (IN2); no longer J3.2
- net U1-GPA7: now also U12.3 (IN1); no longer J3.1
- net U1-GPB0: now also U10.9 (IN4); no longer J3.5
- net U1-GPB1: now also U10.7 (IN3); no longer J3.6
- net U1-GPB2: now also U10.5 (IN2); no longer J2.1
- net U1-GPB3: now also U10.3 (IN1); no longer J2.2
- net U1-GPB4: now also U9.16; no longer J2.3
- net U1-GPB5: now also U9.14; no longer J2.4
- net U1-GPB6: now also U9.12; no longer J2.5
- net U1-GPB7: now also U9.10; no longer J2.6
- new net +24V: C1.1, C2.1, U10.1 (VBB), U10.10 (VBB), U10.11 (VBB), U10.12 (VBB), U10.15 (VBB), U10.16 (VBB), U10.19 (VBB), U10.20 (VBB), U12.1 (VBB), U12.10 (VBB), U12.11 (VBB), U12.12 (VBB), U12.15 (VBB), U12.16 (VBB), U12.19 (VBB), U12.20 (VBB)
- new net ZC57_CLOSE_LED: J2.5, U9.5
- new net ZC57_CLOSE_MOTOR: J2.1, U10.17 (OUT2)
- new net ZC57_OPEN_LED: J2.6, U9.7
- new net ZC57_OPEN_MOTOR: J2.2, U10.18 (OUT1)
- new net ZC58_CLOSE_LED: J2.3, U9.1
- new net ZC58_CLOSE_MOTOR: J3.5, U10.13 (OUT4)
- new net ZC58_OPEN_LED: J2.4, U9.3
- new net ZC58_OPEN_MOTOR: J3.6, U10.14 (OUT3)
- new net ZC59_CLOSE_LED: J3.3, U11.5
- new net ZC59_CLOSE_MOTOR: J4.5, U12.18 (OUT1)
- new net ZC59_OPEN_LED: J3.4, U11.7
- new net ZC59_OPEN_MOTOR: J4.6, U12.17 (OUT2)
- new net ZC60_CLOSE_LED: J3.1, U11.1
- new net ZC60_CLOSE_MOTOR: J4.3, U12.14 (OUT3)
- new net ZC60_OPEN_LED: J3.2, U11.3
- new net ZC60_OPEN_MOTOR: J4.4, U12.13 (OUT4)
Other:
- added sheet relays (relays.kicad_sch)
- moved on the sheet: J2, J3, J4

Commit message: Ekspander update
Connections:
- net GND: no longer C1.2, C2.2, U10.2 (GND1/2), U10.6 (GND3/4), U11.2, U11.4, U11.6, U11.8, U12.2 (GND1/2), U12.6 (GND3/4), U9.2, U9.4, U9.6, U9.8
- new net GNDPWR: C1.2, C2.2, U10.2 (GND1/2), U10.6 (GND3/4), U11.2, U11.4, U11.6, U11.8, U12.2 (GND1/2), U12.6 (GND3/4), U9.2, U9.4, U9.6, U9.8
Changed lines of the file:
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@@
 	(paper "A4")
 	(junction
-		(at 182.88 127)
-		(diameter 0)
-		(color 0 0 0 0)
-	)
-	(junction
 		(at 260.35 92.71)
 		(diameter 0)
@@
 	)
 	(junction
-		(at 240.03 127)
-		(diameter 0)
-		(color 0 0 0 0)
-	)
-	(junction
 		(at 162.56 107.95)
 		(diameter 0)
@@
 	(wire
 		(pts
-			(xy 182.88 127) (xy 182.88 129.54)
-		)
-		(stroke
-			(width 0)
-			(type default)
-		)
-	)
-	(wire
-		(pts
 			(xy 36.83 41.91) (xy 36.83 49.53)
 		)
@@
 	(wire
 		(pts
-			(xy 182.88 123.19) (xy 182.88 127)
+			(xy 182.88 123.19) (xy 182.88 129.54)
 		)
 		(stroke
@@
 	(wire
 		(pts
-			(xy 182.88 127) (xy 240.03 127)
-		)
-		(stroke
-			(width 0)
-			(type default)
-		)
-	)
-	(wire
-		(pts
 			(xy 57.15 72.39) (xy 54.61 72.39)
 		)
@@
 	(wire
 		(pts
-			(xy 240.03 127) (xy 240.03 129.54)
+			(xy 240.03 123.19) (xy 240.03 129.54)
 		)
 		(stroke
@@
 		)
 		(stroke
-			(width 0)
-			(type default)
-		)
-	)
-	(wire
-		(pts
-			(xy 240.03 123.19) (xy 240.03 127)
-		)
-		(stroke

Commit message: ekspander resync
Connections:
- net GNDPWR is gone; now on net GND: C1.2, C2.2, U10.2 (GND1/2), U10.6 (GND3/4), U11.2, U11.4, U11.6, U11.8, U12.2 (GND1/2), U12.6 (GND3/4), U9.2, U9.4, U9.6, U9.8
- net +24V: now also J1.1
- net +5VD renamed +3V3
- net +3V3: no longer J1.1
