File: pcb/espander_100x_i2c/U7.kicad_sch (KiCad schematic)
At the start: 0 parts

Commit message: Resync
Parts:
- added J18, J19, J20, J21: DG127A-5.08-06P-14-00AH, DG127A50806P1400AH, symbol 1_tme:DG127A-5.08-06P-14-00AH
- added U7, U8: MCP23017_SP, Package_DIP:DIP-28_W7.62mm, symbol Interface_Expansion:MCP23017_SP
Connections:
- new net +5VD: U7.9 (VDD), U8.9 (VDD)
- new net GND: U7.10 (VSS), U8.10 (VSS)
- new net SCK: U7.12 (SCK), U8.12 (SCK)
- new net SDA: U7.13 (SDA), U8.13 (SDA)
- new net U7-GPA0: J19.1, U7.21 (GPA0)
- new net U7-GPA1: J19.2, U7.22 (GPA1)
- new net U7-GPA2: J19.3, U7.23 (GPA2)
- new net U7-GPA3: J19.4, U7.24 (GPA3)
- new net U7-GPA4: J19.5, U7.25 (GPA4)
- new net U7-GPA5: J19.6, U7.26 (GPA5)
- new net U7-GPA6: J18.2, U7.27 (GPA6)
- new net U7-GPA7: J18.1, U7.28 (GPA7)
- new net U7-GPB0: J18.3, U7.1 (GPB0)
- new net U7-GPB1: J18.4, U7.2 (GPB1)
- new net U7-GPB2: J18.5, U7.3 (GPB2)
- new net U7-GPB3: J18.6, U7.4 (GPB3)
- new net U7-GPB4: U7.5 (GPB4)
- new net U7-GPB5: U7.6 (GPB5)
- new net U7-GPB6: U7.7 (GPB6)
- new net U7-GPB7: U7.8 (GPB7)
- new net U8-GPA0: U8.21 (GPA0)
- new net U8-GPA1: J21.6, U8.22 (GPA1)
- new net U8-GPA2: J21.1, U8.23 (GPA2)
- new net U8-GPA3: J21.2, U8.24 (GPA3)
- new net U8-GPA4: J21.3, U8.25 (GPA4)
- new net U8-GPA5: J21.4, U8.26 (GPA5)
- new net U8-GPA6: J21.5, U8.27 (GPA6)
- new net U8-GPA7: U8.28 (GPA7)
- new net U8-GPB0: J20.1, U8.1 (GPB0)
- new net U8-GPB1: J20.2, U8.2 (GPB1)
- new net U8-GPB2: J20.3, U8.3 (GPB2)
- new net U8-GPB3: J20.4, U8.4 (GPB3)
- new net U8-GPB4: J20.5, U8.5 (GPB4)
- new net U8-GPB5: J20.6, U8.6 (GPB5)
- new net U8-GPB6: U8.7 (GPB6)
- new net U8-GPB7: U8.8 (GPB7)

Commit message: resync
Connections:
- net U7-GPA0: no longer J19.1
- net U7-GPA1: no longer J19.2
- net U7-GPA2: no longer J19.3
- net U7-GPA3: no longer J19.4
- net U7-GPA4: no longer J19.5
- net U7-GPA5: no longer J19.6
- net U7-GPA6: no longer J18.2
- net U7-GPA7: no longer J18.1
- net U7-GPB0: no longer J18.3
- net U7-GPB1: no longer J18.4
- net U7-GPB2: no longer J18.5
- net U7-GPB3: no longer J18.6
- net U8-GPA1: no longer J21.6
- net U8-GPA2: no longer J21.1
- net U8-GPA3: no longer J21.2
- net U8-GPA4: no longer J21.3
- net U8-GPA5: no longer J21.4
- net U8-GPA6: no longer J21.5
- net U8-GPB0: no longer J20.1
- net U8-GPB1: no longer J20.2
- net U8-GPB2: no longer J20.3
- net U8-GPB3: no longer J20.4
- net U8-GPB4: no longer J20.5
- net U8-GPB5: no longer J20.6
