File: pcb/espander_100x_i2c/U5.kicad_sch (KiCad schematic)
At the start: 0 parts

Commit message: Resync
Parts:
- added J12, J13, J14: DG127A-5.08-06P-14-00AH, DG127A50806P1400AH, symbol 1_tme:DG127A-5.08-06P-14-00AH
- added U5: MCP23017_SP, Package_DIP:DIP-28_W7.62mm, symbol Interface_Expansion:MCP23017_SP
Connections:
- new net +5VD: U5.9 (VDD)
- new net GND: U5.10 (VSS)
- new net SCK: U5.12 (SCK)
- new net SDA: U5.13 (SDA)
- new net U5-GPA0: J14.3, U5.21 (GPA0)
- new net U5-GPA1: J14.4, U5.22 (GPA1)
- new net U5-GPA2: J14.5, U5.23 (GPA2)
- new net U5-GPA3: J14.6, U5.24 (GPA3)
- new net U5-GPA4: J13.4, U5.25 (GPA4)
- new net U5-GPA5: J13.3, U5.26 (GPA5)
- new net U5-GPA6: J13.2, U5.27 (GPA6)
- new net U5-GPA7: J13.1, U5.28 (GPA7)
- new net U5-GPB0: J13.5, U5.1 (GPB0)
- new net U5-GPB1: J13.6, U5.2 (GPB1)
- new net U5-GPB2: J12.1, U5.3 (GPB2)
- new net U5-GPB3: J12.2, U5.4 (GPB3)
- new net U5-GPB4: J12.3, U5.5 (GPB4)
- new net U5-GPB5: J12.4, U5.6 (GPB5)
- new net U5-GPB6: J12.5, U5.7 (GPB6)
- new net U5-GPB7: J12.6, U5.8 (GPB7)
- new net U6-GPB6: J14.1
- new net U6-GPB7: J14.2

Commit message: resync
Connections:
- net U5-GPA0: no longer J14.3
- net U5-GPA1: no longer J14.4
- net U5-GPA2: no longer J14.5
- net U5-GPA3: no longer J14.6
- net U5-GPA4: no longer J13.4
- net U5-GPA5: no longer J13.3
- net U5-GPA6: no longer J13.2
- net U5-GPA7: no longer J13.1
- net U5-GPB0: no longer J13.5
- net U5-GPB1: no longer J13.6
- net U5-GPB2: no longer J12.1
- net U5-GPB3: no longer J12.2
- net U5-GPB4: no longer J12.3
- net U5-GPB5: no longer J12.4
- net U5-GPB6: no longer J12.5
- net U5-GPB7: no longer J12.6
- net U6-GPB6: no longer names the net of J14.1
- net U6-GPB7: no longer names the net of J14.2

Commit message: ekspander resync
Connections:
- net +5VD renamed +3V3
Changed lines of the file:
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@@
 			)
 		)
-		(property "Value" "+5VD"
+		(property "Value" "+3V3"
 			(at 44.704 21.59 0)
 			(effects
