File: pcb/espander_100x_i2c/esp32.kicad_sch (KiCad schematic)
At the start: 2 parts, among them IC1 ESP32-S3-WROOM-1U-N16R8, U9 LTV-847

Commit message: resync
Parts:
- removed U9: LTV-847, Package_DIP:DIP-16_W7.62mm, symbol Isolator:LTV-847

Commit message: ekspander resync
Parts:
- added C3: 10uF, 1_tme:RDEC71H106K3P1H03B, symbol Device:C
- added C4: 100nF, Capacitor_THT:C_Disc_D3.8mm_W2.6mm_P2.50mm, symbol Device:C
- added C5, C6: 22uF, 1_tme:RDEC71H226MWK1H03B, symbol Device:C
- added L1: 4.7uH, 1_tme:LSXND6060YEL4R7NMG, symbol Device:L
- added U13: AP63203WU, Package_TO_SOT_SMD:TSOT-23-6, symbol Regulator_Switching:AP63203WU
Connections:
- net GND: now also C3.2, C5.2, C6.2, U13.4 (GND)
- net +3V3: now reaches IC1.2 (3V3)
- net +3V3: now also C5.1, C6.1, L1.2, U13.1 (FB)
- new net: C4.2, L1.1, U13.6 (BST)
- new net: C4.1, U13.5 (SW)
- new net +24V: C3.1, U13.2 (EN), U13.3 (IN)
