File: pcb/espander_100x_i2c/espander_100x_i2c.kicad_pcb (KiCad board)
At the start: 4 copper layers, 230 x 94 mm, 27 parts, among them J1 DG127A-5.08-06P-14-00AH, J10 DG127A-5.08-06P-14-00AH, J11 DG127A-5.08-06P-14-00AH, J12 DG127A-5.08-06P-14-00AH, J13 DG127A-5.08-06P-14-00AH, J14 DG127A-5.08-06P-14-00AH, J15 DG127A-5.08-06P-14-00AH, J16 DG127A-5.08-06P-14-00AH, J17 DG127A-5.08-06P-14-00AH, J18 DG127A-5.08-06P-14-00AH, J19 DG127A-5.08-06P-14-00AH, J2 DG127A-5.08-06P-14-00AH, J20 DG127A-5.08-06P-14-00AH, J3 DG127A-5.08-06P-14-00AH, J4 DG127A-5.08-06P-14-00AH, J5 DG127A-5.08-06P-14-00AH, J6 DG127A-5.08-06P-14-00AH, J7 DG127A-5.08-06P-14-00AH, J8 DG127A-5.08-06P-14-00AH, J9 DG127A-5.08-06P-14-00AH, U1 MCP23017_SP, U2 MCP23017_SP, U3 MCP23017_SP, U4 MCP23017_SP, U5 MCP23017_SP, U6 MCP23017_SP, U7 MCP23017_SP

Commit message: Add initial DRU file for espander_100x_i2c PCB design
Parts:
- removed J11, J12, J13, J14, J15, J16, J17, J18, J19, J20: DG127A-5.08-06P-14-00AH, 1_tme:DG127A50806P1400AH
- removed U5, U6, U7: MCP23017_SP, Package_DIP:DIP-28_W7.62mm
- moved U4 55.9 mm to (188.0, 36.5)
- moved J8 44.4 mm to (144.9, 18.1)
- moved J5 44.4 mm to (80.9, 18.1)
- moved J9 44.3 mm to (166.3, 18.1)
- moved J6 44.3 mm to (102.3, 18.1)
- moved J10 44.3 mm to (187.6, 18.1)
- moved J7 44.2 mm to (123.7, 18.1)
- moved U3 37.5 mm to (141.9, 36.4)
- moved U1 30.7 mm to (41.0, 36.4)
- moved J2 29.8 mm to (29.1, 28.2), turned to 180 degrees
- moved J3 29.7 mm to (50.5, 28.2), turned to 180 degrees
- moved J4 29.6 mm to (71.9, 28.2), turned to 180 degrees
- moved U2 29.1 mm to (105.3, 36.4)
- moved J1 24.3 mm to (28.1, 57.0), turned to -90 degrees
Connections:
- J1 pad 1: Net-(U1-GPB0) -> +5VD
- J1 pad 2: Net-(U1-GPB1) -> GND
- J1 pad 3: Net-(U1-GPB2) -> unconnected-(J1-Pad3)
- J1 pad 4: Net-(U1-GPB3) -> unconnected-(J1-Pad4)
- J1 pad 5: Net-(U1-GPB4) -> SDA
- J1 pad 6: Net-(U1-GPB5) -> SCK
- J2 pad 1: unconnected-(J2-Pad1) -> /U1-GPB2
- J2 pad 2: unconnected-(J2-Pad2) -> /U1-GPB3
- J2 pad 3: unconnected-(J2-Pad3) -> /U1-GPB4
- J2 pad 4: unconnected-(J2-Pad4) -> /U1-GPB5
- J2 pad 5: unconnected-(J2-Pad5) -> /U1-GPB6
- J2 pad 6: unconnected-(J2-Pad6) -> /U1-GPB7
- J3 pad 1: unconnected-(J3-Pad1) -> /U1-GPA7
- J3 pad 2: unconnected-(J3-Pad2) -> /U1-GPA6
- J3 pad 3: unconnected-(J3-Pad3) -> /U1-GPA5
- J3 pad 4: unconnected-(J3-Pad4) -> /U1-GPA4
- J3 pad 5: unconnected-(J3-Pad5) -> /U1-GPB0
- J3 pad 6: unconnected-(J3-Pad6) -> /U1-GPB1
- J4 pad 1: unconnected-(J4-Pad1) -> U2-GPB6
- J4 pad 2: unconnected-(J4-Pad2) -> U2-GPB7
- J4 pad 3: unconnected-(J4-Pad3) -> /U1-GPA0
- J4 pad 4: unconnected-(J4-Pad4) -> /U1-GPA1
- J4 pad 5: unconnected-(J4-Pad5) -> /U1-GPA2
- J4 pad 6: unconnected-(J4-Pad6) -> /U1-GPA3
- J5 pad 1: unconnected-(J5-Pad1) -> /U2/U2-GPB5
- J5 pad 2: unconnected-(J5-Pad2) -> /U2/U2-GPB4
- J5 pad 3: unconnected-(J5-Pad3) -> /U2/U2-GPB3
- J5 pad 4: unconnected-(J5-Pad4) -> /U2/U2-GPB2
- J5 pad 5: unconnected-(J5-Pad5) -> /U2/U2-GPB1
- J5 pad 6: unconnected-(J5-Pad6) -> /U2/U2-GPB0
- J6 pad 1: unconnected-(J6-Pad1) -> /U2/U2-GPA0
- J6 pad 2: unconnected-(J6-Pad2) -> /U2/U2-GPA1
- J6 pad 3: unconnected-(J6-Pad3) -> /U2/U2-GPA2
- J6 pad 4: unconnected-(J6-Pad4) -> /U2/U2-GPA3
- J6 pad 5: unconnected-(J6-Pad5) -> /U2/U2-GPA4
- J6 pad 6: unconnected-(J6-Pad6) -> /U2/U2-GPA5
- J7 pad 1: unconnected-(J7-Pad1) -> /U2/U2-GPA7
- J7 pad 2: unconnected-(J7-Pad2) -> /U2/U2-GPA6
- J7 pad 3: unconnected-(J7-Pad3) -> U3-GPB7
- J7 pad 4: unconnected-(J7-Pad4) -> U3-GPB6
- J7 pad 5: unconnected-(J7-Pad5) -> U3-GPB5
- J7 pad 6: unconnected-(J7-Pad6) -> U3-GPB4
- J8 pad 1: unconnected-(J8-Pad1) -> /U3/U3-GPB0
- J8 pad 2: unconnected-(J8-Pad2) -> /U3/U3-GPB1
- J8 pad 3: unconnected-(J8-Pad3) -> /U3/U3-GPB2
- J8 pad 4: unconnected-(J8-Pad4) -> /U3/U3-GPB3
- J8 pad 5: unconnected-(J8-Pad5) -> /U3/U3-GPA7
- J8 pad 6: unconnected-(J8-Pad6) -> /U3/U3-GPA6
- J9 pad 1: unconnected-(J9-Pad1) -> /U3/U3-GPA5
- J9 pad 2: unconnected-(J9-Pad2) -> /U3/U3-GPA4
- J9 pad 3: unconnected-(J9-Pad3) -> /U3/U3-GPA3
- J9 pad 4: unconnected-(J9-Pad4) -> /U3/U3-GPA2
- J9 pad 5: unconnected-(J9-Pad5) -> /U3/U3-GPA1
- J9 pad 6: unconnected-(J9-Pad6) -> /U3/U3-GPA0
- U1 pad 1: Net-(U1-GPB0) -> /U1-GPB0
- U1 pad 10: Net-(U1-VSS) -> GND
- U1 pad 12: Net-(U1-SCK) -> SCK
- U1 pad 13: Net-(U1-SDA) -> SDA
- U1 pad 2: Net-(U1-GPB1) -> /U1-GPB1
- U1 pad 21: Net-(U1-GPA0) -> /U1-GPA0
- U1 pad 22: Net-(U1-GPA1) -> /U1-GPA1
- U1 pad 23: Net-(U1-GPA2) -> /U1-GPA2
- U1 pad 24: Net-(U1-GPA3) -> /U1-GPA3
- U1 pad 25: unconnected-(U1-GPA4-Pad25) -> /U1-GPA4
- U1 pad 26: unconnected-(U1-GPA5-Pad26) -> /U1-GPA5
- U1 pad 27: unconnected-(U1-GPA6-Pad27) -> /U1-GPA6
- U1 pad 28: unconnected-(U1-GPA7-Pad28) -> /U1-GPA7
- U1 pad 3: Net-(U1-GPB2) -> /U1-GPB2
- U1 pad 4: Net-(U1-GPB3) -> /U1-GPB3
- U1 pad 5: Net-(U1-GPB4) -> /U1-GPB4
- U1 pad 6: Net-(U1-GPB5) -> /U1-GPB5
- U1 pad 7: Net-(U1-GPB6) -> /U1-GPB6
- U1 pad 8: /<NO NET> -> /U1-GPB7
- U1 pad 9: Net-(U1-VDD) -> +5VD
- U2 pad 1: unconnected-(U2-GPB0-Pad1) -> /U2/U2-GPB0
- U2 pad 10: Net-(U1-VSS) -> GND
- U2 pad 12: Net-(U1-SCK) -> SCK
- U2 pad 13: Net-(U1-SDA) -> SDA
- U2 pad 2: unconnected-(U2-GPB1-Pad2) -> /U2/U2-GPB1
- U2 pad 21: unconnected-(U2-GPA0-Pad21) -> /U2/U2-GPA0
- U2 pad 22: unconnected-(U2-GPA1-Pad22) -> /U2/U2-GPA1
- U2 pad 23: unconnected-(U2-GPA2-Pad23) -> /U2/U2-GPA2
- U2 pad 24: unconnected-(U2-GPA3-Pad24) -> /U2/U2-GPA3
- U2 pad 25: unconnected-(U2-GPA4-Pad25) -> /U2/U2-GPA4
- U2 pad 26: unconnected-(U2-GPA5-Pad26) -> /U2/U2-GPA5
- U2 pad 27: unconnected-(U2-GPA6-Pad27) -> /U2/U2-GPA6
- U2 pad 28: unconnected-(U2-GPA7-Pad28) -> /U2/U2-GPA7
- U2 pad 3: unconnected-(U2-GPB2-Pad3) -> /U2/U2-GPB2
- U2 pad 4: unconnected-(U2-GPB3-Pad4) -> /U2/U2-GPB3
- U2 pad 5: unconnected-(U2-GPB4-Pad5) -> /U2/U2-GPB4
- U2 pad 6: unconnected-(U2-GPB5-Pad6) -> /U2/U2-GPB5
- U2 pad 7: unconnected-(U2-GPB6-Pad7) -> U2-GPB6
- U2 pad 8: unconnected-(U2-GPB7-Pad8) -> U2-GPB7
- U2 pad 9: Net-(U1-VDD) -> +5VD
- U3 pad 1: unconnected-(U3-GPB0-Pad1) -> /U3/U3-GPB0
- U3 pad 10: Net-(U1-VSS) -> GND
- U3 pad 12: Net-(U1-SCK) -> SCK
- U3 pad 13: Net-(U1-SDA) -> SDA
- U3 pad 2: unconnected-(U3-GPB1-Pad2) -> /U3/U3-GPB1
- U3 pad 21: unconnected-(U3-GPA0-Pad21) -> /U3/U3-GPA0
- U3 pad 22: unconnected-(U3-GPA1-Pad22) -> /U3/U3-GPA1
- U3 pad 23: unconnected-(U3-GPA2-Pad23) -> /U3/U3-GPA2
- U3 pad 24: unconnected-(U3-GPA3-Pad24) -> /U3/U3-GPA3
- U3 pad 25: unconnected-(U3-GPA4-Pad25) -> /U3/U3-GPA4
- U3 pad 26: unconnected-(U3-GPA5-Pad26) -> /U3/U3-GPA5
- U3 pad 27: unconnected-(U3-GPA6-Pad27) -> /U3/U3-GPA6
- U3 pad 28: unconnected-(U3-GPA7-Pad28) -> /U3/U3-GPA7
- U3 pad 3: unconnected-(U3-GPB2-Pad3) -> /U3/U3-GPB2
- U3 pad 4: unconnected-(U3-GPB3-Pad4) -> /U3/U3-GPB3
- U3 pad 5: unconnected-(U3-GPB4-Pad5) -> U3-GPB4
- U3 pad 6: unconnected-(U3-GPB5-Pad6) -> U3-GPB5
- U3 pad 7: unconnected-(U3-GPB6-Pad7) -> U3-GPB6
- U3 pad 8: unconnected-(U3-GPB7-Pad8) -> U3-GPB7
- U3 pad 9: Net-(U1-VDD) -> +5VD
- U4 pad 1: unconnected-(U4-GPB0-Pad1) -> /U3/U4-GPB0
- U4 pad 10: Net-(U1-VSS) -> GND
- U4 pad 12: Net-(U1-SCK) -> SCK
- U4 pad 13: Net-(U1-SDA) -> SDA
- U4 pad 2: unconnected-(U4-GPB1-Pad2) -> /U3/U4-GPB1
- U4 pad 21: unconnected-(U4-GPA0-Pad21) -> /U3/U4-GPA0
- U4 pad 22: unconnected-(U4-GPA1-Pad22) -> /U3/U4-GPA1
- U4 pad 23: unconnected-(U4-GPA2-Pad23) -> /U3/U4-GPA2
- U4 pad 24: unconnected-(U4-GPA3-Pad24) -> /U3/U4-GPA3
- U4 pad 25: unconnected-(U4-GPA4-Pad25) -> /U3/U4-GPA4
- U4 pad 26: unconnected-(U4-GPA5-Pad26) -> /U3/U4-GPA5
- U4 pad 27: unconnected-(U4-GPA6-Pad27) -> /U3/U4-GPA6
- U4 pad 28: unconnected-(U4-GPA7-Pad28) -> /U3/U4-GPA7
- U4 pad 3: unconnected-(U4-GPB2-Pad3) -> /U3/U4-GPB2
- U4 pad 4: unconnected-(U4-GPB3-Pad4) -> /U3/U4-GPB3
- U4 pad 5: unconnected-(U4-GPB4-Pad5) -> U4-GPB4
- U4 pad 6: unconnected-(U4-GPB5-Pad6) -> U4-GPB5
- U4 pad 7: unconnected-(U4-GPB6-Pad7) -> U4-GPB6
- U4 pad 8: unconnected-(U4-GPB7-Pad8) -> U4-GPB7
- U4 pad 9: Net-(U1-VDD) -> +5VD
Routing:
- net Net-(U1-GPA3): track 166.3 -> 0.00 mm
- net Net-(U1-SCK): track 157.5 -> 0.00 mm
- net Net-(U1-VSS): track 156.7 -> 0.00 mm
- net Net-(U1-VDD): track 156.0 -> 0.00 mm
- net Net-(U1-SDA): track 155.4 -> 0.00 mm
- net Net-(U1-GPA2): track 92.4 -> 0.00 mm
- net Net-(U1-GPA1): track 72.6 -> 0.00 mm
- net U2-GPB7: track 0.00 -> 58.4 mm
- net /<NO NET>: track 50.1 -> 0.00 mm
- net /U3/U3-GPA1: track 0.00 -> 47.3 mm
- net Net-(U1-GPB5): track 46.5 -> 0.00 mm
- net /U1-GPB7: track 0.00 -> 46.4 mm
- net Net-(U1-GPA0): track 45.5 -> 0.00 mm
- net U2-GPB6: track 0.00 -> 44.3 mm
- net Net-(U1-GPB6): track 44.0 -> 0.00 mm
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Other:
- board outline removed

Commit message: Refactor code structure for improved readability and maintainability
Parts:
- added J11: DG127A-5.08-06P-14-00AH, 1_tme:DG127A50806P1400AH, F.Cu at (221.2, 28.2)
- moved J8 15.9 mm to (157.2, 28.2), turned to 180 degrees
- moved J9 15.9 mm to (178.5, 28.2), turned to 180 degrees
- moved J5 15.9 mm to (93.1, 28.2), turned to 180 degrees
- moved J10 15.9 mm to (199.8, 28.2), turned to 180 degrees
- moved J6 15.8 mm to (114.5, 28.2), turned to 180 degrees
- moved J7 15.8 mm to (135.8, 28.2), turned to 180 degrees
- moved U3 7.20 mm to (149.0, 37.1)
- moved U2 7.05 mm to (98.3, 36.9)
- moved U4 3.53 mm to (191.4, 37.1)
- moved J4 0.09 mm to (71.8, 28.2)
- moved J3 0.06 mm to (50.5, 28.2)
Connections:
- net /U3/U4-GPA0 renamed /U3 - U4/U4-GPA0
- net /U3/U4-GPA1 renamed /U3 - U4/U4-GPA1
- net /U3/U4-GPA2 renamed /U3 - U4/U4-GPA2
- net /U3/U4-GPA3 renamed /U3 - U4/U4-GPA3
- net /U3/U4-GPA4 renamed /U3 - U4/U4-GPA4
- net /U3/U4-GPA5 renamed /U3 - U4/U4-GPA5
- net /U3/U4-GPA6 renamed /U3 - U4/U4-GPA6
- net /U3/U4-GPA7 renamed /U3 - U4/U4-GPA7
- net /U3/U4-GPB0 renamed /U3 - U4/U4-GPB0
- net /U3/U4-GPB1 renamed /U3 - U4/U4-GPB1
- net /U3/U4-GPB2 renamed /U3 - U4/U4-GPB2
- net /U3/U4-GPB3 renamed /U3 - U4/U4-GPB3
- net U4-GPB4 renamed /U3 - U4/U4-GPB4
- net U4-GPB5 renamed /U3 - U4/U4-GPB5
- net U4-GPB6 renamed /U3 - U4/U4-GPB6
- net U4-GPB7 renamed /U3 - U4/U4-GPB7
- J5 pad 1: /U2/U2-GPB5 -> /U2/U2-GPB0
- J5 pad 2: /U2/U2-GPB4 -> /U2/U2-GPB1
- J5 pad 3: /U2/U2-GPB3 -> /U2/U2-GPB2
- J5 pad 4: /U2/U2-GPB2 -> /U2/U2-GPB3
- J5 pad 5: /U2/U2-GPB1 -> /U2/U2-GPB4
- J5 pad 6: /U2/U2-GPB0 -> /U2/U2-GPB5
- J6 pad 1: /U2/U2-GPA0 -> /U2/U2-GPA4
- J6 pad 2: /U2/U2-GPA1 -> /U2/U2-GPA5
- J6 pad 3: /U2/U2-GPA2 -> /U2/U2-GPA6
- J6 pad 4: /U2/U2-GPA3 -> /U2/U2-GPA7
- J6 pad 5: /U2/U2-GPA4 -> /U2/U2-GPA1
- J6 pad 6: /U2/U2-GPA5 -> /U2/U2-GPA0
- J7 pad 1: /U2/U2-GPA7 -> unconnected-(J7-Pad1)
- J7 pad 2: /U2/U2-GPA6 -> unconnected-(J7-Pad2)
- J7 pad 3: U3-GPB7 -> unconnected-(J7-Pad3)
- J7 pad 4: U3-GPB6 -> unconnected-(J7-Pad4)
- J7 pad 5: U3-GPB5 -> /U2/U2-GPA2
- J7 pad 6: U3-GPB4 -> /U2/U2-GPA3
- J8 pad 1: /U3/U3-GPB0 -> unconnected-(J8-Pad1)
- J8 pad 2: /U3/U3-GPB1 -> unconnected-(J8-Pad2)
- J8 pad 3: /U3/U3-GPB2 -> unconnected-(J8-Pad3)
- J8 pad 4: /U3/U3-GPB3 -> unconnected-(J8-Pad4)
- J8 pad 5: /U3/U3-GPA7 -> unconnected-(J8-Pad5)
- J8 pad 6: /U3/U3-GPA6 -> unconnected-(J8-Pad6)
- J9 pad 1: /U3/U3-GPA5 -> unconnected-(J9-Pad1)
- J9 pad 2: /U3/U3-GPA4 -> unconnected-(J9-Pad2)
- J9 pad 3: /U3/U3-GPA3 -> unconnected-(J9-Pad3)
- J9 pad 4: /U3/U3-GPA2 -> unconnected-(J9-Pad4)
- J9 pad 5: /U3/U3-GPA1 -> unconnected-(J9-Pad5)
- J9 pad 6: /U3/U3-GPA0 -> unconnected-(J9-Pad6)
- U3 pad 1: /U3/U3-GPB0 -> /U3 - U4/U3-GPB0
- U3 pad 2: /U3/U3-GPB1 -> /U3 - U4/U3-GPB1
- U3 pad 21: /U3/U3-GPA0 -> /U3 - U4/U3-GPA0
- U3 pad 22: /U3/U3-GPA1 -> /U3 - U4/U3-GPA1
- U3 pad 23: /U3/U3-GPA2 -> /U3 - U4/U3-GPA2
- U3 pad 24: /U3/U3-GPA3 -> /U3 - U4/U3-GPA3
- U3 pad 25: /U3/U3-GPA4 -> /U3 - U4/U3-GPA4
- U3 pad 26: /U3/U3-GPA5 -> /U3 - U4/U3-GPA5
- U3 pad 27: /U3/U3-GPA6 -> /U3 - U4/U3-GPA6
- U3 pad 28: /U3/U3-GPA7 -> /U3 - U4/U3-GPA7
- U3 pad 3: /U3/U3-GPB2 -> /U3 - U4/U3-GPB2
- U3 pad 4: /U3/U3-GPB3 -> /U3 - U4/U3-GPB3
Routing:
- net SCK: track 0.00 -> 153.1 mm
- net /U3/U3-GPA1: track 47.3 -> 0.00 mm
- net U3-GPB7: track 41.1 -> 0.00 mm
- net /U3/U3-GPA0: track 40.8 -> 0.00 mm
- net /U3/U3-GPA3: track 39.9 -> 0.00 mm
- net U3-GPB5: track 34.0 -> 0.00 mm
- net /U3/U3-GPA2: track 33.5 -> 0.00 mm
- net /U3/U3-GPA5: track 32.4 -> 0.00 mm
- net U3-GPB6: track 27.4 -> 0.00 mm
- net /U3/U3-GPB2: track 26.3 -> 0.00 mm
- net /U3/U3-GPA4: track 26.1 -> 0.00 mm
- net /U3/U3-GPB0: track 21.2 -> 0.00 mm
- net /U3/U3-GPA7: track 20.2 -> 0.00 mm
- net U3-GPB4: track 20.2 -> 0.00 mm
- net /U3/U3-GPB3: track 19.8 -> 0.00 mm
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Other:
- board outline added: 500 x 100 mm

Commit message: RESYNC
Parts:
- moved J1 195.8 mm to (222.9, 77.0)
Connections:
- J7 pad 1: unconnected-(J7-Pad1) -> U3-GPB4
- J7 pad 2: unconnected-(J7-Pad2) -> U3-GPB5
- J7 pad 3: unconnected-(J7-Pad3) -> U3-GPB6
- J7 pad 4: unconnected-(J7-Pad4) -> U3-GPB7
- J8 pad 1: unconnected-(J8-Pad1) -> /U3 - U4/U3-GPA7
- J8 pad 2: unconnected-(J8-Pad2) -> /U3 - U4/U3-GPA6
- J8 pad 3: unconnected-(J8-Pad3) -> /U3 - U4/U3-GPB0
- J8 pad 4: unconnected-(J8-Pad4) -> /U3 - U4/U3-GPB1
- J8 pad 5: unconnected-(J8-Pad5) -> /U3 - U4/U3-GPB2
- J8 pad 6: unconnected-(J8-Pad6) -> /U3 - U4/U3-GPB3
- J9 pad 1: unconnected-(J9-Pad1) -> /U3 - U4/U3-GPA0
- J9 pad 2: unconnected-(J9-Pad2) -> /U3 - U4/U3-GPA1
- J9 pad 3: unconnected-(J9-Pad3) -> /U3 - U4/U3-GPA2
- J9 pad 4: unconnected-(J9-Pad4) -> /U3 - U4/U3-GPA3
- J9 pad 5: unconnected-(J9-Pad5) -> /U3 - U4/U3-GPA4
- J9 pad 6: unconnected-(J9-Pad6) -> /U3 - U4/U3-GPA5
- U3 pad 5: U3-GPB4 -> /U3 - U4/U3-GPB4
- U3 pad 6: U3-GPB5 -> /U3 - U4/U3-GPB5
- U3 pad 7: U3-GPB6 -> /U3 - U4/U3-GPB6
- U3 pad 8: U3-GPB7 -> /U3 - U4/U3-GPB7
Routing:
- net U3-GPB7: track 0.00 -> 45.5 mm
- net /U3 - U4/U3-GPA1: track 0.00 -> 42.3 mm
- net U3-GPB5: track 0.00 -> 38.3 mm
- net /U3 - U4/U3-GPA0: track 0.00 -> 35.8 mm
- net /U3 - U4/U3-GPA3: track 0.00 -> 35.1 mm
- net U3-GPB6: track 0.00 -> 31.8 mm
- net /U3 - U4/U3-GPB3: track 0.00 -> 28.6 mm
- net /U3 - U4/U3-GPA2: track 0.00 -> 28.6 mm
- net /U3 - U4/U3-GPA5: track 0.00 -> 28.0 mm
- net U3-GPB4: track 0.00 -> 24.6 mm
- net /U3 - U4/U3-GPB1: track 0.00 -> 23.1 mm
- net /U3 - U4/U3-GPA6: track 0.00 -> 22.5 mm
- net /U3 - U4/U3-GPA4: track 0.00 -> 21.4 mm
- net /U3 - U4/U3-GPB2: track 0.00 -> 15.7 mm
- net /U3 - U4/U3-GPB0: track 0.00 -> 10.2 mm
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Other:
- board text added: "DLA GPIO xxA7 i xxB7 MOGĄ BYĆ TYLKO JAKO WYJŚCIE W PRZYPADKU KONTROLERA MCP23017"
- board text added: "U1B7 | U1B5 | U1B3 U1B6 | U1B4 | UB2"

Commit message: Resync
Parts:
- added IC1: ESP32-S3-WROOM-1U-N16R8, 1_tme:ESP32S3WROOM1UN16R8, F.Cu at (234.4, 91.2)
- added J12: DG127A-5.08-06P-14-00AH, 1_tme:DG127A50806P1400AH, F.Cu at (244.1, 28.2)
- added J13: DG127A-5.08-06P-14-00AH, 1_tme:DG127A50806P1400AH, F.Cu at (265.6, 28.2)
- added J14: DG127A-5.08-06P-14-00AH, 1_tme:DG127A50806P1400AH, F.Cu at (287.1, 28.2)
- added J15: DG127A-5.08-06P-14-00AH, 1_tme:DG127A50806P1400AH, F.Cu at (308.3, 28.2)
- added J16: DG127A-5.08-06P-14-00AH, 1_tme:DG127A50806P1400AH, F.Cu at (329.5, 28.2)
- added J17: DG127A-5.08-06P-14-00AH, 1_tme:DG127A50806P1400AH, F.Cu at (351.3, 28.2)
- added J18: DG127A-5.08-06P-14-00AH, 1_tme:DG127A50806P1400AH, F.Cu at (373.2, 28.2)
- added J19: DG127A-5.08-06P-14-00AH, 1_tme:DG127A50806P1400AH, F.Cu at (394.7, 28.2)
- added J20: DG127A-5.08-06P-14-00AH, 1_tme:DG127A50806P1400AH, F.Cu at (416.2, 28.2)
- added J21: DG127A-5.08-06P-14-00AH, 1_tme:DG127A50806P1400AH, F.Cu at (437.7, 28.2)
- added U5: MCP23017_SP, Package_DIP:DIP-28_W7.62mm, F.Cu at (256.0, 36.9)
- added U6: MCP23017_SP, Package_DIP:DIP-28_W7.62mm, F.Cu at (309.6, 36.7)
- added U7: MCP23017_SP, Package_DIP:DIP-28_W7.62mm, F.Cu at (363.2, 36.8)
- added U8: MCP23017_SP, Package_DIP:DIP-28_W7.62mm, F.Cu at (416.8, 36.8)
- added U9: LTV-847, Package_DIP:DIP-16_W7.62mm, F.Cu at (20.2, 50.6)
- moved J1 251.4 mm to (473.1, 52.7), turned to 0 degrees
- moved U4 9.23 mm to (200.7, 37.0)
- moved J11 1.48 mm to (222.6, 28.2)
- moved J10 1.31 mm to (201.1, 28.2)
- moved J9 1.15 mm to (179.6, 28.2)
- moved J8 0.98 mm to (158.1, 28.2)
- moved J7 0.82 mm to (136.6, 28.2)
- moved J6 0.66 mm to (115.1, 28.2)
- moved J5 0.49 mm to (93.6, 28.2)
- moved J4 0.33 mm to (72.1, 28.2)
- moved J3 0.16 mm to (50.6, 28.2)
Connections:
- J10 pad 1: unconnected-(J10-Pad1) -> /U3 - U4/U4-GPB0
- J10 pad 2: unconnected-(J10-Pad2) -> /U3 - U4/U4-GPB1
- J10 pad 3: unconnected-(J10-Pad3) -> /U3 - U4/U4-GPB2
- J10 pad 4: unconnected-(J10-Pad4) -> /U3 - U4/U4-GPB3
- J10 pad 5: unconnected-(J10-Pad5) -> /U3 - U4/U4-GPB4
- J10 pad 6: unconnected-(J10-Pad6) -> /U3 - U4/U4-GPB5
- J11 pad 1: unconnected-(J11-Pad1) -> /U3 - U4/U4-GPA2
- J11 pad 2: unconnected-(J11-Pad2) -> /U3 - U4/U4-GPA3
- J11 pad 3: unconnected-(J11-Pad3) -> /U3 - U4/U4-GPA4
- J11 pad 4: unconnected-(J11-Pad4) -> /U3 - U4/U4-GPA5
- J11 pad 5: unconnected-(J11-Pad5) -> /U3 - U4/U4-GPA6
- J11 pad 6: unconnected-(J11-Pad6) -> /U3 - U4/U4-GPA1
- U3 pad 5: /U3 - U4/U3-GPB4 -> U3-GPB4
- U3 pad 6: /U3 - U4/U3-GPB5 -> U3-GPB5
- U3 pad 7: /U3 - U4/U3-GPB6 -> U3-GPB6
- U3 pad 8: /U3 - U4/U3-GPB7 -> U3-GPB7
Routing:
- net SCK: track 153.1 -> 58.1 mm
- net U6-GPB7: track 0.00 -> 46.8 mm
- net /U5/U5-GPB7: track 0.00 -> 46.8 mm
- net U7-GPB7: track 0.00 -> 44.7 mm
- net /U7 - U8/U7-GPA1: track 0.00 -> 42.8 mm
- net /U5/U5-GPA1: track 0.00 -> 40.7 mm
- net /U5/U5-GPB5: track 0.00 -> 39.6 mm
- net /U6/U6-GPA0: track 0.00 -> 39.3 mm
- net /U3 - U4/U4-GPB5: track 0.00 -> 37.8 mm
- net /U6/U6-GPA3: track 0.00 -> 37.7 mm
- net U7-GPB5: track 0.00 -> 37.5 mm
- net /U6/U6-GPB5: track 0.00 -> 37.2 mm
- net /U7 - U8/U8-GPB5: track 0.00 -> 37.0 mm
- net /U7 - U8/U8-GPA1: track 0.00 -> 36.9 mm
- net /U3 - U4/U4-GPA1: track 0.00 -> 36.4 mm
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Other:
- board text added: "U1A3 | U1A1 | U1B7 U1A2 | U1A0 | U1B6"
- board text added: "U1B1 | U1B4 | U1B6 U1B0 | U1B5 | U1B7"
- board text added: "U1B7 | U1B5 | U1B3 U1B6 | U1B4 | U1B2"
- board text removed: "U1B7 | U1B5 | U1B3 U1B6 | U1B4 | UB2"

Commit message: resync
Parts:
- added C1: 100nF, Capacitor_THT:C_Disc_D3.0mm_W2.0mm_P2.50mm, F.Cu at (20.1, 49.5)
- added C2: 100nF, Capacitor_THT:C_Disc_D3.0mm_W2.0mm_P2.50mm, F.Cu at (59.9, 45.6)
- added K1: G5Q-1A, Relay_THT:Relay_SPST_Omron-G5Q-1A, F.Cu at (-76.8, 243.6)
- added K10: G5Q-1A, Relay_THT:Relay_SPST_Omron-G5Q-1A, F.Cu at (36.3, 243.6)
- added K11: G5Q-1A, Relay_THT:Relay_SPST_Omron-G5Q-1A, F.Cu at (48.9, 243.6)
- added K12: G5Q-1A, Relay_THT:Relay_SPST_Omron-G5Q-1A, F.Cu at (61.4, 243.6)
- added K13: G5Q-1A, Relay_THT:Relay_SPST_Omron-G5Q-1A, F.Cu at (74.0, 243.6)
- added K14: G5Q-1A, Relay_THT:Relay_SPST_Omron-G5Q-1A, F.Cu at (86.6, 243.6)
- added K15: G5Q-1A, Relay_THT:Relay_SPST_Omron-G5Q-1A, F.Cu at (99.1, 243.6)
- added K16: G5Q-1A, Relay_THT:Relay_SPST_Omron-G5Q-1A, F.Cu at (111.7, 243.6)
- added K17: G5Q-1A, Relay_THT:Relay_SPST_Omron-G5Q-1A, F.Cu at (124.3, 243.6)
- added K18: G5Q-1A, Relay_THT:Relay_SPST_Omron-G5Q-1A, F.Cu at (136.9, 243.6)
- added K19: G5Q-1A, Relay_THT:Relay_SPST_Omron-G5Q-1A, F.Cu at (149.4, 243.6)
- added K2: G5Q-1A, Relay_THT:Relay_SPST_Omron-G5Q-1A, F.Cu at (-64.3, 243.6)
- added K20: G5Q-1A, Relay_THT:Relay_SPST_Omron-G5Q-1A, F.Cu at (162.0, 243.6)
- added K21: G5Q-1A, Relay_THT:Relay_SPST_Omron-G5Q-1A, F.Cu at (174.6, 243.6)
- added K22: G5Q-1A, Relay_THT:Relay_SPST_Omron-G5Q-1A, F.Cu at (187.1, 243.6)
- added K23: G5Q-1A, Relay_THT:Relay_SPST_Omron-G5Q-1A, F.Cu at (199.7, 243.6)
- added K24: G5Q-1A, Relay_THT:Relay_SPST_Omron-G5Q-1A, F.Cu at (212.3, 243.6)
- added K25: G5Q-1A, Relay_THT:Relay_SPST_Omron-G5Q-1A, F.Cu at (224.9, 243.6)
- added K26: G5Q-1A, Relay_THT:Relay_SPST_Omron-G5Q-1A, F.Cu at (237.4, 243.6)
- added K27: G5Q-1A, Relay_THT:Relay_SPST_Omron-G5Q-1A, F.Cu at (250.0, 243.6)
- added K28: G5Q-1A, Relay_THT:Relay_SPST_Omron-G5Q-1A, F.Cu at (262.6, 243.6)
- added K29: G5Q-1A, Relay_THT:Relay_SPST_Omron-G5Q-1A, F.Cu at (275.1, 243.6)
- added K3: G5Q-1A, Relay_THT:Relay_SPST_Omron-G5Q-1A, F.Cu at (-51.7, 243.6)
- added K30: G5Q-1A, Relay_THT:Relay_SPST_Omron-G5Q-1A, F.Cu at (287.7, 243.6)
- added K31: G5Q-1A, Relay_THT:Relay_SPST_Omron-G5Q-1A, F.Cu at (300.3, 243.6)
- added K32: G5Q-1A, Relay_THT:Relay_SPST_Omron-G5Q-1A, F.Cu at (312.8, 243.6)
- added K33: G5Q-1A, Relay_THT:Relay_SPST_Omron-G5Q-1A, F.Cu at (325.4, 243.6)
- added K34: G5Q-1A, Relay_THT:Relay_SPST_Omron-G5Q-1A, F.Cu at (338.0, 243.6)
- added K35: G5Q-1A, Relay_THT:Relay_SPST_Omron-G5Q-1A, F.Cu at (350.6, 243.6)
- added K36: G5Q-1A, Relay_THT:Relay_SPST_Omron-G5Q-1A, F.Cu at (363.1, 243.6)
- added K37: G5Q-1A, Relay_THT:Relay_SPST_Omron-G5Q-1A, F.Cu at (375.7, 243.6)
- added K38: G5Q-1A, Relay_THT:Relay_SPST_Omron-G5Q-1A, F.Cu at (388.3, 243.6)
- added K39: G5Q-1A, Relay_THT:Relay_SPST_Omron-G5Q-1A, F.Cu at (400.8, 243.6)
- added K4: G5Q-1A, Relay_THT:Relay_SPST_Omron-G5Q-1A, F.Cu at (-39.1, 243.6)
- added K40: G5Q-1A, Relay_THT:Relay_SPST_Omron-G5Q-1A, F.Cu at (413.4, 243.6)
- added K41: G5Q-1A, Relay_THT:Relay_SPST_Omron-G5Q-1A, F.Cu at (426.0, 243.6)
- added K42: G5Q-1A, Relay_THT:Relay_SPST_Omron-G5Q-1A, F.Cu at (438.6, 243.6)
- added K43: G5Q-1A, Relay_THT:Relay_SPST_Omron-G5Q-1A, F.Cu at (451.1, 243.6)
- added K44: G5Q-1A, Relay_THT:Relay_SPST_Omron-G5Q-1A, F.Cu at (463.7, 243.6)
- added K45: G5Q-1A, Relay_THT:Relay_SPST_Omron-G5Q-1A, F.Cu at (476.3, 243.6)
- added K46: G5Q-1A, Relay_THT:Relay_SPST_Omron-G5Q-1A, F.Cu at (488.8, 243.6)
- added K47: G5Q-1A, Relay_THT:Relay_SPST_Omron-G5Q-1A, F.Cu at (501.4, 243.6)
- added K48: G5Q-1A, Relay_THT:Relay_SPST_Omron-G5Q-1A, F.Cu at (514.0, 243.6)
- added K49: G5Q-1A, Relay_THT:Relay_SPST_Omron-G5Q-1A, F.Cu at (526.5, 243.6)
- added K5: G5Q-1A, Relay_THT:Relay_SPST_Omron-G5Q-1A, F.Cu at (-26.6, 243.6)
- added K50: G5Q-1A, Relay_THT:Relay_SPST_Omron-G5Q-1A, F.Cu at (539.1, 243.6)
- added K6: G5Q-1A, Relay_THT:Relay_SPST_Omron-G5Q-1A, F.Cu at (-14.0, 243.6)
- added K7: G5Q-1A, Relay_THT:Relay_SPST_Omron-G5Q-1A, F.Cu at (-1.41, 243.6)
- added K8: G5Q-1A, Relay_THT:Relay_SPST_Omron-G5Q-1A, F.Cu at (11.2, 243.6)
- added K9: G5Q-1A, Relay_THT:Relay_SPST_Omron-G5Q-1A, F.Cu at (23.7, 243.6)
- added U10: ITS716G, Package_SO:SOIC-20W_7.5x12.8mm_P1.27mm, F.Cu at (27.9, 40.8)
- added U11: LTV-847, Package_DIP:DIP-16_W7.62mm, F.Cu at (56.1, 37.0)
- added U12: ITS716G, Package_SO:SOIC-20W_7.5x12.8mm_P1.27mm, F.Cu at (68.2, 40.6)
- moved IC1 258.7 mm to (482.4, 17.6)
- moved U1 15.8 mm to (41.3, 52.2)
- moved U9 7.72 mm to (15.2, 56.5)
Connections:
- J10 pad 1: /U3 - U4/U4-GPB0 -> unconnected-(J10-Pad1)
- J10 pad 2: /U3 - U4/U4-GPB1 -> unconnected-(J10-Pad2)
- J10 pad 3: /U3 - U4/U4-GPB2 -> unconnected-(J10-Pad3)
- J10 pad 4: /U3 - U4/U4-GPB3 -> unconnected-(J10-Pad4)
- J10 pad 5: /U3 - U4/U4-GPB4 -> unconnected-(J10-Pad5)
- J10 pad 6: /U3 - U4/U4-GPB5 -> unconnected-(J10-Pad6)
- J11 pad 1: /U3 - U4/U4-GPA2 -> unconnected-(J11-Pad1)
- J11 pad 2: /U3 - U4/U4-GPA3 -> unconnected-(J11-Pad2)
- J11 pad 3: /U3 - U4/U4-GPA4 -> unconnected-(J11-Pad3)
- J11 pad 4: /U3 - U4/U4-GPA5 -> unconnected-(J11-Pad4)
- J11 pad 5: /U3 - U4/U4-GPA6 -> unconnected-(J11-Pad5)
- J11 pad 6: /U3 - U4/U4-GPA1 -> unconnected-(J11-Pad6)
- J12 pad 1: /U5/U5-GPB2 -> unconnected-(J12-Pad1)
- J12 pad 2: /U5/U5-GPB3 -> unconnected-(J12-Pad2)
- J12 pad 3: /U5/U5-GPB4 -> unconnected-(J12-Pad3)
- J12 pad 4: /U5/U5-GPB5 -> unconnected-(J12-Pad4)
- J12 pad 5: /U5/U5-GPB6 -> unconnected-(J12-Pad5)
- J12 pad 6: /U5/U5-GPB7 -> unconnected-(J12-Pad6)
- J13 pad 1: /U5/U5-GPA7 -> unconnected-(J13-Pad1)
- J13 pad 2: /U5/U5-GPA6 -> unconnected-(J13-Pad2)
- J13 pad 3: /U5/U5-GPA5 -> unconnected-(J13-Pad3)
- J13 pad 4: /U5/U5-GPA4 -> unconnected-(J13-Pad4)
- J13 pad 5: /U5/U5-GPB0 -> unconnected-(J13-Pad5)
- J13 pad 6: /U5/U5-GPB1 -> unconnected-(J13-Pad6)
- J14 pad 1: U6-GPB6 -> unconnected-(J14-Pad1)
- J14 pad 2: U6-GPB7 -> unconnected-(J14-Pad2)
- J14 pad 3: /U5/U5-GPA0 -> unconnected-(J14-Pad3)
- J14 pad 4: /U5/U5-GPA1 -> unconnected-(J14-Pad4)
- J14 pad 5: /U5/U5-GPA2 -> unconnected-(J14-Pad5)
- J14 pad 6: /U5/U5-GPA3 -> unconnected-(J14-Pad6)
- J15 pad 1: /U6/U6-GPB0 -> unconnected-(J15-Pad1)
- J15 pad 2: /U6/U6-GPB1 -> unconnected-(J15-Pad2)
- J15 pad 3: /U6/U6-GPB2 -> unconnected-(J15-Pad3)
- J15 pad 4: /U6/U6-GPB3 -> unconnected-(J15-Pad4)
- J15 pad 5: /U6/U6-GPB4 -> unconnected-(J15-Pad5)
- J15 pad 6: /U6/U6-GPB5 -> unconnected-(J15-Pad6)
- J16 pad 1: /U6/U6-GPA4 -> unconnected-(J16-Pad1)
- J16 pad 2: /U6/U6-GPA5 -> unconnected-(J16-Pad2)
- J16 pad 3: /U6/U6-GPA6 -> unconnected-(J16-Pad3)
- J16 pad 4: /U6/U6-GPA7 -> unconnected-(J16-Pad4)
- J16 pad 5: /U6/U6-GPA1 -> unconnected-(J16-Pad5)
- J16 pad 6: /U6/U6-GPA0 -> unconnected-(J16-Pad6)
- J17 pad 1: U7-GPB4 -> unconnected-(J17-Pad1)
- J17 pad 2: U7-GPB5 -> unconnected-(J17-Pad2)
- J17 pad 3: U7-GPB6 -> unconnected-(J17-Pad3)
- J17 pad 4: U7-GPB7 -> unconnected-(J17-Pad4)
- J17 pad 5: /U6/U6-GPA2 -> unconnected-(J17-Pad5)
- J17 pad 6: /U6/U6-GPA3 -> unconnected-(J17-Pad6)
- J18 pad 1: /U7 - U8/U7-GPA7 -> unconnected-(J18-Pad1)
- J18 pad 2: /U7 - U8/U7-GPA6 -> unconnected-(J18-Pad2)
- J18 pad 3: /U7 - U8/U7-GPB0 -> unconnected-(J18-Pad3)
- J18 pad 4: /U7 - U8/U7-GPB1 -> unconnected-(J18-Pad4)
- J18 pad 5: /U7 - U8/U7-GPB2 -> unconnected-(J18-Pad5)
- J18 pad 6: /U7 - U8/U7-GPB3 -> unconnected-(J18-Pad6)
- J19 pad 1: /U7 - U8/U7-GPA0 -> unconnected-(J19-Pad1)
- J19 pad 2: /U7 - U8/U7-GPA1 -> unconnected-(J19-Pad2)
- J19 pad 3: /U7 - U8/U7-GPA2 -> unconnected-(J19-Pad3)
- J19 pad 4: /U7 - U8/U7-GPA3 -> unconnected-(J19-Pad4)
- J19 pad 5: /U7 - U8/U7-GPA4 -> unconnected-(J19-Pad5)
- J19 pad 6: /U7 - U8/U7-GPA5 -> unconnected-(J19-Pad6)
- J2 pad 1: /U1-GPB2 -> /ZC57_CLOSE_MOTOR
- J2 pad 2: /U1-GPB3 -> /ZC57_OPEN_MOTOR
- J2 pad 3: /U1-GPB4 -> /ZC58_CLOSE_LED
- J2 pad 4: /U1-GPB5 -> /ZC58_OPEN_LED
- J2 pad 5: /U1-GPB6 -> /ZC57_CLOSE_LED
- J2 pad 6: /U1-GPB7 -> /ZC57_OPEN_LED
- J20 pad 1: /U7 - U8/U8-GPB0 -> unconnected-(J20-Pad1)
- J20 pad 2: /U7 - U8/U8-GPB1 -> unconnected-(J20-Pad2)
- J20 pad 3: /U7 - U8/U8-GPB2 -> unconnected-(J20-Pad3)
- J20 pad 4: /U7 - U8/U8-GPB3 -> unconnected-(J20-Pad4)
- J20 pad 5: /U7 - U8/U8-GPB4 -> unconnected-(J20-Pad5)
- J20 pad 6: /U7 - U8/U8-GPB5 -> unconnected-(J20-Pad6)
- J21 pad 1: /U7 - U8/U8-GPA2 -> unconnected-(J21-Pad1)
- J21 pad 2: /U7 - U8/U8-GPA3 -> unconnected-(J21-Pad2)
- J21 pad 3: /U7 - U8/U8-GPA4 -> unconnected-(J21-Pad3)
- J21 pad 4: /U7 - U8/U8-GPA5 -> unconnected-(J21-Pad4)
- J21 pad 5: /U7 - U8/U8-GPA6 -> unconnected-(J21-Pad5)
- J21 pad 6: /U7 - U8/U8-GPA1 -> unconnected-(J21-Pad6)
- J3 pad 1: /U1-GPA7 -> /ZC60_CLOSE_LED
- J3 pad 2: /U1-GPA6 -> /ZC60_OPEN_LED
- J3 pad 3: /U1-GPA5 -> /ZC59_CLOSE_LED
- J3 pad 4: /U1-GPA4 -> /ZC59_OPEN_LED
- J3 pad 5: /U1-GPB0 -> /ZC58_CLOSE_MOTOR
- J3 pad 6: /U1-GPB1 -> /ZC58_OPEN_MOTOR
- J4 pad 3: /U1-GPA0 -> /ZC60_CLOSE_MOTOR
- J4 pad 4: /U1-GPA1 -> /ZC60_OPEN_MOTOR
- J4 pad 5: /U1-GPA2 -> /ZC59_CLOSE_MOTOR
- J4 pad 6: /U1-GPA3 -> /ZC59_OPEN_MOTOR
- J5 pad 1: /U2/U2-GPB0 -> unconnected-(J5-Pad1)
- J5 pad 2: /U2/U2-GPB1 -> unconnected-(J5-Pad2)
- J5 pad 3: /U2/U2-GPB2 -> unconnected-(J5-Pad3)
- J5 pad 4: /U2/U2-GPB3 -> unconnected-(J5-Pad4)
- J5 pad 5: /U2/U2-GPB4 -> unconnected-(J5-Pad5)
- J5 pad 6: /U2/U2-GPB5 -> unconnected-(J5-Pad6)
- J6 pad 1: /U2/U2-GPA4 -> unconnected-(J6-Pad1)
- J6 pad 2: /U2/U2-GPA5 -> unconnected-(J6-Pad2)
- J6 pad 3: /U2/U2-GPA6 -> unconnected-(J6-Pad3)
- J6 pad 4: /U2/U2-GPA7 -> unconnected-(J6-Pad4)
- J6 pad 5: /U2/U2-GPA1 -> unconnected-(J6-Pad5)
- J6 pad 6: /U2/U2-GPA0 -> unconnected-(J6-Pad6)
- J7 pad 1: U3-GPB4 -> unconnected-(J7-Pad1)
- J7 pad 2: U3-GPB5 -> unconnected-(J7-Pad2)
- J7 pad 3: U3-GPB6 -> unconnected-(J7-Pad3)
- J7 pad 4: U3-GPB7 -> unconnected-(J7-Pad4)
- J7 pad 5: /U2/U2-GPA2 -> unconnected-(J7-Pad5)
- J7 pad 6: /U2/U2-GPA3 -> unconnected-(J7-Pad6)
- J8 pad 1: /U3 - U4/U3-GPA7 -> unconnected-(J8-Pad1)
- J8 pad 2: /U3 - U4/U3-GPA6 -> unconnected-(J8-Pad2)
- J8 pad 3: /U3 - U4/U3-GPB0 -> unconnected-(J8-Pad3)
- J8 pad 4: /U3 - U4/U3-GPB1 -> unconnected-(J8-Pad4)
- J8 pad 5: /U3 - U4/U3-GPB2 -> unconnected-(J8-Pad5)
- J8 pad 6: /U3 - U4/U3-GPB3 -> unconnected-(J8-Pad6)
- J9 pad 1: /U3 - U4/U3-GPA0 -> unconnected-(J9-Pad1)
- J9 pad 2: /U3 - U4/U3-GPA1 -> unconnected-(J9-Pad2)
- J9 pad 3: /U3 - U4/U3-GPA2 -> unconnected-(J9-Pad3)
- J9 pad 4: /U3 - U4/U3-GPA3 -> unconnected-(J9-Pad4)
- J9 pad 5: /U3 - U4/U3-GPA4 -> unconnected-(J9-Pad5)
- J9 pad 6: /U3 - U4/U3-GPA5 -> unconnected-(J9-Pad6)
- U2 pad 7: U2-GPB6 -> /U2/U2-GPB6
- U2 pad 8: U2-GPB7 -> /U2/U2-GPB7
- U9 pad 1: unconnected-(U9-Pad1) -> /ZC58_CLOSE_LED
- U9 pad 10: unconnected-(U9-Pad10) -> /U1-GPB7
- U9 pad 11: unconnected-(U9-Pad11) -> GND
- U9 pad 12: unconnected-(U9-Pad12) -> /U1-GPB6
- U9 pad 13: unconnected-(U9-Pad13) -> GND
- U9 pad 14: unconnected-(U9-Pad14) -> /U1-GPB5
- U9 pad 15: unconnected-(U9-Pad15) -> GND
- U9 pad 16: unconnected-(U9-Pad16) -> /U1-GPB4
- U9 pad 2: unconnected-(U9-Pad2) -> GND
- U9 pad 3: unconnected-(U9-Pad3) -> /ZC58_OPEN_LED
- U9 pad 4: unconnected-(U9-Pad4) -> GND
- U9 pad 5: unconnected-(U9-Pad5) -> /ZC57_CLOSE_LED
- U9 pad 6: unconnected-(U9-Pad6) -> GND
- U9 pad 7: unconnected-(U9-Pad7) -> /ZC57_OPEN_LED
- U9 pad 8: unconnected-(U9-Pad8) -> GND
- U9 pad 9: unconnected-(U9-Pad9) -> GND
Routing:
- net SCK: track 58.1 -> 0.00 mm
- net U2-GPB7: track 50.2 -> 0.00 mm
- net U6-GPB7: track 46.8 -> 0.00 mm
- net /U5/U5-GPB7: track 46.8 -> 0.00 mm
- net U3-GPB7: track 45.2 -> 0.00 mm
- net U7-GPB7: track 44.7 -> 0.00 mm
- net /U7 - U8/U7-GPA1: track 42.8 -> 0.00 mm
- net /U3 - U4/U3-GPA1: track 42.8 -> 0.00 mm
- net /U5/U5-GPA1: track 40.7 -> 0.00 mm
- net /U5/U5-GPB5: track 39.6 -> 0.00 mm
- net /U6/U6-GPA0: track 39.3 -> 0.00 mm
- net /U2/U2-GPB5: track 38.9 -> 0.00 mm
- net /U2/U2-GPA0: track 38.3 -> 0.00 mm
- net U3-GPB5: track 38.0 -> 0.00 mm
- net /U3 - U4/U4-GPB5: track 37.8 -> 0.00 mm
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- added copper zone on F.Cu, net +24V
- added copper zone on B.Cu, net GND
