File: pcb/espander_100x_i2c/espander_100x_i2c.kicad_pcb (KiCad board)
At the start: 4 copper layers, 500 x 100 mm, 86 parts, among them IC1 ESP32-S3-WROOM-1U-N16R8, J1 DG127A-5.08-06P-14-00AH, J10 DG127A-5.08-06P-14-00AH, J11 DG127A-5.08-06P-14-00AH, J12 DG127A-5.08-06P-14-00AH, J13 DG127A-5.08-06P-14-00AH, J14 DG127A-5.08-06P-14-00AH, J15 DG127A-5.08-06P-14-00AH, J16 DG127A-5.08-06P-14-00AH, J17 DG127A-5.08-06P-14-00AH, J18 DG127A-5.08-06P-14-00AH, J19 DG127A-5.08-06P-14-00AH, J2 DG127A-5.08-06P-14-00AH, J20 DG127A-5.08-06P-14-00AH, J21 DG127A-5.08-06P-14-00AH, J3 DG127A-5.08-06P-14-00AH, J4 DG127A-5.08-06P-14-00AH, J5 DG127A-5.08-06P-14-00AH, J6 DG127A-5.08-06P-14-00AH, J7 DG127A-5.08-06P-14-00AH, J8 DG127A-5.08-06P-14-00AH, J9 DG127A-5.08-06P-14-00AH, K1 G5Q-1A, K10 G5Q-1A, K11 G5Q-1A, K12 G5Q-1A, K13 G5Q-1A, K14 G5Q-1A, K15 G5Q-1A, K16 G5Q-1A, K17 G5Q-1A, K18 G5Q-1A, K19 G5Q-1A, K2 G5Q-1A, K20 G5Q-1A, K21 G5Q-1A, K22 G5Q-1A, K23 G5Q-1A, K24 G5Q-1A, K25 G5Q-1A, K26 G5Q-1A, K27 G5Q-1A, K28 G5Q-1A, K29 G5Q-1A, K3 G5Q-1A, K30 G5Q-1A, K31 G5Q-1A, K32 G5Q-1A, K33 G5Q-1A, K34 G5Q-1A, K35 G5Q-1A, K36 G5Q-1A, K37 G5Q-1A, K38 G5Q-1A, K39 G5Q-1A, K4 G5Q-1A, K40 G5Q-1A, K41 G5Q-1A, K42 G5Q-1A, K43 G5Q-1A, K44 G5Q-1A, K45 G5Q-1A, K46 G5Q-1A, K47 G5Q-1A, K48 G5Q-1A, K49 G5Q-1A, K5 G5Q-1A, K50 G5Q-1A, K6 G5Q-1A, K7 G5Q-1A, K8 G5Q-1A, K9 G5Q-1A, U1 MCP23017_SP, U10 ITS716G, U11 LTV-847, U12 ITS716G, U2 MCP23017_SP, U3 MCP23017_SP, U4 MCP23017_SP, U5 MCP23017_SP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

Commit message: gitignore#2
Parts:
- moved C1 0.95 mm to (21.0, 49.5)
Routing:
- net /ZC58_CLOSE_LED: track 0.00 -> 57.0 mm
- net /ZC57_OPEN_LED: track 0.00 -> 55.6 mm
- net /ZC58_OPEN_LED: track 0.00 -> 46.1 mm
- net /ZC57_CLOSE_LED: track 0.00 -> 40.0 mm
Changed lines of the file:
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@@
 	(footprint "Capacitor_THT:C_Disc_D3.0mm_W2.0mm_P2.50mm"
 		(layer "F.Cu")
-		(at 20.05 49.45)
+		(at 21 49.5)
 		(descr "C, Disc series, Radial, pin pitch=2.50mm, diameter*width=3*2mm^2, Capacitor")
 		(tags "C Disc series Radial pin pitch 2.50mm diameter 3mm width 2mm Capacitor")
@@
 	)
 	(segment
+		(start 23.5 48.69)
+		(end 23.5 49.5)
+		(width 1)
+		(layer "F.Cu")
+		(net 9)
+	)
+	(segment
+		(start 23.405 48.595)
+		(end 23.5 48.69)
+		(width 1)
+		(layer "F.Cu")
+		(net 9)
+	)
+	(segment
 		(start 62.9 48.1)
 		(end 63.755 47.245)
@@
 	)
 	(segment
-		(start 23.405 48.595)
-		(end 22.55 49.45)
-		(width 1)
-		(layer "F.Cu")
-		(net 9)
-	)
-	(segment
 		(start 23.405 45.4)
 		(end 23.405 48.595)
@@
 	)
 	(segment
+		(start 21 48.5)
+		(end 21 49.5)
+		(width 1)
+		(layer "F.Cu")
+		(net 441)
+	)
+	(segment
 		(start 22.135 47.365)
-		(end 20.05 49.45)
+		(end 21 48.5)
 		(width 1)
 		(layer "F.Cu")
@@
 	)
 	(segment
+		(start 13.5 70.005)
+		(end 13.5 20.98)
+		(width 0.3048)
+		(layer "F.Cu")
+		(net 442)
+	)
+	(segment
+		(start 15.245 71.75)
+		(end 13.5 70.005)
+		(width 0.3048)
+		(layer "F.Cu")
+		(net 442)
+	)
+	(segment
+		(start 13.5 20.98)
+		(end 16.43 18.05)
+		(width 0.3048)
+		(layer "F.Cu")
+		(net 442)
+	)
+	(segment
+		(start 18.5 63.415)
+		(end 18.5 28.68)
+		(width 0.3048)
+		(layer "F.Cu")
+		(net 443)
+	)
+	(segment
+		(start 15.245 66.67)
+		(end 18.5 63.415)
+		(width 0.3048)
+		(layer "F.Cu")
+		(net 443)
+	)
+	(segment
+		(start 18.5 28.68)
+		(end 18.97 28.21)
+		(width 0.3048)
+		(layer "F.Cu")
+		(net 443)
+	)
+	(segment
 		(start 24.675 32.075)
 		(end 26.59 30.16)
@@
 	)
 	(segment
+		(start 17 22.56)
+		(end 21.51 18.05)
+		(width 0.3048)
+		(layer "F.Cu")
+		(net 445)
+	)
+	(segment
+		(start 17 59.835)
+		(end 17 22.56)
+		(width 0.3048)
+		(layer "F.Cu")
+		(net 445)
+	)
+	(segment
+		(start 15.245 61.59)
+		(end 17 59.835)
+		(width 0.3048)
+		(layer "F.Cu")
+		(net 445)
+	)
+	(segment
+		(start 21 16)
+		(end 22 16)
+		(width 0.3048)
+		(layer "F.Cu")
+		(net 446)
+	)
+	(segment
+		(start 24.05 18.05)
+		(end 24.05 28.21)
+		(width 0.3048)
+		(layer "F.Cu")
+		(net 446)
+	)
+	(segment
+		(start 22 16)
+		(end 24.05 18.05)
+		(width 0.3048)
+		(layer "F.Cu")
+		(net 446)
+	)
+	(segment
+		(start 15.245 21.755)
+		(end 21 16)
+		(width 0.3048)
+		(layer "F.Cu")
+		(net 446)
+	)
+	(segment
+		(start 15.245 56.51)
+		(end 15.245 21.755)
+		(width 0.3048)
+		(layer "F.Cu")
+		(net 446)
+	)
+	(segment

Commit message: ekspander resync
Parts:
- added C3: 10uF, 1_tme:RDEC71H106K3P1H03B, F.Cu at (455.8, 19.6)
- added C4: 100nF, Capacitor_THT:C_Disc_D3.8mm_W2.6mm_P2.50mm, F.Cu at (465.9, 18.6)
- added C5: 22uF, 1_tme:RDEC71H226MWK1H03B, F.Cu at (478.8, 12.4)
- added C6: 22uF, 1_tme:RDEC71H226MWK1H03B, F.Cu at (478.8, 18.8)
- added L1: 4.7uH, 1_tme:LSXND6060YEL4R7NMG, F.Cu at (472.1, 15.6)
- added U13: AP63203WU, Package_TO_SOT_SMD:TSOT-23-6, F.Cu at (461.4, 18.3)
- moved IC1 19.7 mm to (499.1, 28.1), turned to -90 degrees
Connections:
- IC1 pad 2: unconnected-(IC1-3V3-Pad2) -> +3V3
- J1 pad 1: +5VD -> +24V
- U1 pad 9: +5VD -> +3V3
- U2 pad 9: +5VD -> +3V3
- U3 pad 9: +5VD -> +3V3
- U4 pad 9: +5VD -> +3V3
- U5 pad 9: +5VD -> +3V3
- U6 pad 9: +5VD -> +3V3
- U7 pad 9: +5VD -> +3V3
- U8 pad 9: +5VD -> +3V3
Routing:
- net +3V3: track 0.00 -> 18.1 mm
- net +24V: track 7.35 -> 12.9 mm
- net Net-(U13-BST): track 0.00 -> 3.83 mm
- net Net-(U13-SW): track 0.00 -> 3.44 mm
- added copper zone on F.Cu, net +3V3
