File: pcb/arduino_nano/ardiuno_nano/ardiuno_nano.kicad_pcb (KiCad board)
At the start: 2 copper layers, 43.2 x 17.8 mm, 8 parts, among them J1 Analog, J2 Digital, U1 MCP23017_SO

Commit message: Refactor code structure and remove redundant sections for improved readability and maintainability
Parts:
- removed A1: Arduino_Nano_Every, Module:Arduino_Nano
- removed U1: MCP23017_SO, Package_SO:SOIC-28W_7.5x17.9mm_P1.27mm
Other:
- board outline removed
- board text removed: "ICSP"
- board text removed: "USB Mini-B"
