File: pcb/arduino_nano/ardiuno_nano/ardiuno_nano.kicad_sch (KiCad schematic)
At the start: 2 parts, among them J1 Analog, J2 Digital

Commit message: Refactor code structure and remove redundant sections for improved readability and maintainability
Parts:
- added A1: Arduino_Nano_Every, Module:Arduino_Nano, symbol MCU_Module:Arduino_Nano_Every
- added U1: MCP23017_SO, Package_SO:SOIC-28W_7.5x17.9mm_P1.27mm, symbol Interface_Expansion:MCP23017_SO
Connections:
- new net: A1.23 (SDA/A4), U1.13 (SDA)
- new net: A1.24 (SCL/A5), U1.12 (SCK)
- new net: A1.29 (GND), A1.4 (GND)
