File: pcb/ekspander_100x_i2c/ekspander_100x_i2c.kicad_pcb (KiCad board)
At the start: 4 copper layers, 500 x 100 mm, 92 parts, among them IC1 ESP32-S3-WROOM-1U-N16R8, J1 DG127A-5.08-06P-14-00AH, J10 DG127A-5.08-06P-14-00AH, J11 DG127A-5.08-06P-14-00AH, J12 DG127A-5.08-06P-14-00AH, J13 DG127A-5.08-06P-14-00AH, J14 DG127A-5.08-06P-14-00AH, J15 DG127A-5.08-06P-14-00AH, J16 DG127A-5.08-06P-14-00AH, J17 DG127A-5.08-06P-14-00AH, J18 DG127A-5.08-06P-14-00AH, J19 DG127A-5.08-06P-14-00AH, J2 DG127A-5.08-06P-14-00AH, J20 DG127A-5.08-06P-14-00AH, J21 DG127A-5.08-06P-14-00AH, J3 DG127A-5.08-06P-14-00AH, J4 DG127A-5.08-06P-14-00AH, J5 DG127A-5.08-06P-14-00AH, J6 DG127A-5.08-06P-14-00AH, J7 DG127A-5.08-06P-14-00AH, J8 DG127A-5.08-06P-14-00AH, J9 DG127A-5.08-06P-14-00AH, K1 G5Q-1A, K10 G5Q-1A, K11 G5Q-1A, K12 G5Q-1A, K13 G5Q-1A, K14 G5Q-1A, K15 G5Q-1A, K16 G5Q-1A, K17 G5Q-1A, K18 G5Q-1A, K19 G5Q-1A, K2 G5Q-1A, K20 G5Q-1A, K21 G5Q-1A, K22 G5Q-1A, K23 G5Q-1A, K24 G5Q-1A, K25 G5Q-1A, K26 G5Q-1A, K27 G5Q-1A, K28 G5Q-1A, K29 G5Q-1A, K3 G5Q-1A, K30 G5Q-1A, K31 G5Q-1A, K32 G5Q-1A, K33 G5Q-1A, K34 G5Q-1A, K35 G5Q-1A, K36 G5Q-1A, K37 G5Q-1A, K38 G5Q-1A, K39 G5Q-1A, K4 G5Q-1A, K40 G5Q-1A, K41 G5Q-1A, K42 G5Q-1A, K43 G5Q-1A, K44 G5Q-1A, K45 G5Q-1A, K46 G5Q-1A, K47 G5Q-1A, K48 G5Q-1A, K49 G5Q-1A, K5 G5Q-1A, K50 G5Q-1A, K6 G5Q-1A, K7 G5Q-1A, K8 G5Q-1A, K9 G5Q-1A, U1 MCP23017_SP, U10 ITS716G, U11 LTV-847, U12 ITS716G, U13 AP63203WU, U2 MCP23017_SP, U3 MCP23017_SP, U4 MCP23017_SP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

Commit message: Ekspander 100x - zasilanie 3V3
Parts:
- added C7: 1uF_50V, Capacitor_THT:C_Disc_D5.0mm_W2.5mm_P5.00mm, F.Cu at (245.3, 90.2)
- added C8: 22uF, 1_tme:RDEC71H226MWK1H03B, F.Cu at (253.4, 93.5)
- added C9: 0.1uF, 1_tme:RDEC71H226MWK1H03B, F.Cu at (247.3, 93.5)
- added R1: 10K, 1_tme:RESAD1520W50L600D230, F.Cu at (260.2, 86.9)
- moved IC1 274.5 mm to (232.0, 91.4), turned to 180 degrees
- moved C5 224.3 mm to (270.1, 94.7), turned to 180 degrees
- moved C6 220.0 mm to (270.1, 88.4), turned to 180 degrees
- moved L1 209.5 mm to (276.9, 91.6), turned to 180 degrees
- moved C4 195.8 mm to (283.0, 88.5), turned to -90 degrees
- moved U13 187.7 mm to (287.5, 88.9), turned to 180 degrees
- moved C3 176.6 mm to (293.1, 88.2), turned to 90 degrees
- moved C1 0.15 mm to (20.9, 49.5)
Connections:
- IC1 pad 13: unconnected-(IC1-IO19-Pad13) -> /esp32/USB_D_N
- IC1 pad 14: unconnected-(IC1-IO20-Pad14) -> /esp32/USB_D_P
- IC1 pad 3: unconnected-(IC1-EN-Pad3) -> Net-(IC1-EN)
- IC1 pad 4: unconnected-(IC1-IO4-Pad4) -> /esp32/SDA
- IC1 pad 5: unconnected-(IC1-IO5-Pad5) -> /esp32/SCK
Routing:
- net +3V3: track 18.1 -> 91.2 mm
- net Net-(IC1-EN): track 0.00 -> 13.8 mm
- net +24V: track 12.9 -> 1.00 mm
- net GND: track 11.6 -> 16.7 mm, vias 0 -> 56
- net /ZC58_CLOSE_LED: track 57.0 -> 58.4 mm
- added copper zone on F.Cu, net GND

Commit message: Ekspander U2 - U3 - U4 update
Parts:
- added C10: 0.1uF, Capacitor_SMD:C_0805_2012Metric_Pad1.18x1.45mm_HandSolder, F.Cu at (61.6, 85.8)
- added C11: 0.1uF, Capacitor_SMD:C_0805_2012Metric_Pad1.18x1.45mm_HandSolder, F.Cu at (69.5, 79.9)
- added C12: 0.1uF, Capacitor_SMD:C_0805_2012Metric_Pad1.18x1.45mm_HandSolder, F.Cu at (69.5, 82.9)
- added C13: 0.1uF, Capacitor_SMD:C_0805_2012Metric_Pad1.18x1.45mm_HandSolder, F.Cu at (69.5, 87.9)
- added C14: 0.1uF, Capacitor_SMD:C_0805_2012Metric_Pad1.18x1.45mm_HandSolder, F.Cu at (69.5, 93.0)
- added C15: 0.1uF, Capacitor_SMD:C_0805_2012Metric_Pad1.18x1.45mm_HandSolder, F.Cu at (69.5, 71.9)
- added C16: 0.1uF, Capacitor_SMD:C_0805_2012Metric_Pad1.18x1.45mm_HandSolder, F.Cu at (69.5, 74.9)
- added C17: 0.1uF, Capacitor_SMD:C_0805_2012Metric_Pad1.18x1.45mm_HandSolder, F.Cu at (87.2, 47.8)
- added C18: 0.1uF, Capacitor_SMD:C_0805_2012Metric_Pad1.18x1.45mm_HandSolder, F.Cu at (145.8, 48.0)
- added C19: 0.1uF, Capacitor_SMD:C_0805_2012Metric_Pad1.18x1.45mm_HandSolder, F.Cu at (125.3, 47.8)
- added C20: 0.1uF, Capacitor_SMD:C_0805_2012Metric_Pad1.18x1.45mm_HandSolder, F.Cu at (174.1, 48.4)
- added U14: LTV-847, Package_DIP:DIP-16_W7.62mm, F.Cu at (77.9, 53.8)
- added U15: ITS716G, Package_SO:SOIC-20W_7.5x12.8mm_P1.27mm, F.Cu at (92.2, 40.1)
- added U16: ITS716G, Package_SO:SOIC-20W_7.5x12.8mm_P1.27mm, F.Cu at (131.2, 40.2)
- added U17: LTV-847, Package_DIP:DIP-16_W7.62mm, F.Cu at (119.5, 36.5)
- added U18: LTV-847, Package_DIP:DIP-16_W7.62mm, F.Cu at (143.2, 54.0)
- added U19: LTV-847, Package_DIP:DIP-16_W7.62mm, F.Cu at (161.4, 35.4)
- added U20: LTV-847, Package_DIP:DIP-16_W7.62mm, F.Cu at (194.0, 63.1)
- added U21: ITS716G, Package_SO:SOIC-20W_7.5x12.8mm_P1.27mm, F.Cu at (151.7, 40.5)
- added U22: ITS716G, Package_SO:SOIC-20W_7.5x12.8mm_P1.27mm, F.Cu at (180.1, 40.6)
- C3: footprint 1_tme:RDEC71H106K3P1H03B -> Capacitor_SMD:C_0805_2012Metric_Pad1.18x1.45mm_HandSolder
- C4: footprint Capacitor_THT:C_Disc_D3.8mm_W2.6mm_P2.50mm -> Capacitor_SMD:C_0805_2012Metric_Pad1.18x1.45mm_HandSolder
- C5, C6, C8, C9: footprint 1_tme:RDEC71H226MWK1H03B -> Capacitor_SMD:C_0805_2012Metric_Pad1.18x1.45mm_HandSolder
- C7: footprint Capacitor_THT:C_Disc_D5.0mm_W2.5mm_P5.00mm -> Capacitor_SMD:C_0805_2012Metric_Pad1.18x1.45mm_HandSolder
- R1: footprint 1_tme:RESAD1520W50L600D230 -> PCM_Resistor_SMD_AKL:R_0805_2012Metric_Pad1.20x1.40mm_HandSolder
- moved J1 192.2 mm to (283.9, 86.6)
- moved U4 34.4 mm to (235.0, 38.5)
- moved U3 30.0 mm to (172.5, 55.8)
- moved C3 17.1 mm to (276.4, 92.2)
- moved U2 16.0 mm to (96.7, 52.8)
- moved R1 15.9 mm to (248.4, 97.5), turned to 90 degrees
- moved U13 15.2 mm to (273.1, 93.8)
- moved C4 14.8 mm to (269.5, 94.5)
- moved C6 13.2 mm to (257.3, 91.5)
- moved L1 13.1 mm to (263.9, 93.4)
- moved C5 12.9 mm to (257.3, 95.3)
- moved C8 9.58 mm to (246.1, 99.7), turned to 90 degrees
- moved C7 8.42 mm to (252.0, 95.3)
- moved C9 7.09 mm to (243.8, 99.7), turned to 90 degrees
Connections:
- IC1 pad 4: /esp32/SDA -> SDA
- IC1 pad 5: /esp32/SCK -> SCK
- J4 pad 1: U2-GPB6 -> ZC61_CLOSE_LED
- J4 pad 2: U2-GPB7 -> ZC61_OPEN_LED
- J5 pad 1: unconnected-(J5-Pad1) -> /U2/ZC62_CLOSE_MOTOR
- J5 pad 2: unconnected-(J5-Pad2) -> /U2/ZC62_OPEN_MOTOR
- J5 pad 3: unconnected-(J5-Pad3) -> /U2/ZC61_CLOSE_MOTOR
- J5 pad 4: unconnected-(J5-Pad4) -> /U2/ZC61_OPEN_MOTOR
- J5 pad 5: unconnected-(J5-Pad5) -> /U2/ZC62_OPEN_LED
- J5 pad 6: unconnected-(J5-Pad6) -> /U2/ZC62_CLOSE_LED
- J6 pad 1: unconnected-(J6-Pad1) -> /U2/ZC63_CLOSE_MOTOR
- J6 pad 2: unconnected-(J6-Pad2) -> /U2/ZC63_OPEN_MOTOR
- J6 pad 3: unconnected-(J6-Pad3) -> /U2/ZC63_CLOSE_LED
- J6 pad 4: unconnected-(J6-Pad4) -> /U2/ZC63_OPEN_LED
- J6 pad 5: unconnected-(J6-Pad5) -> /U2/ZC64_CLOSE_LED
- J6 pad 6: unconnected-(J6-Pad6) -> /U2/ZC64_OPEN_LED
- J7 pad 1: unconnected-(J7-Pad1) -> /U2/ZC65_OPEN_LED
- J7 pad 2: unconnected-(J7-Pad2) -> /U2/ZC65_CLOSE_LED
- J7 pad 3: unconnected-(J7-Pad3) -> /U2/ZC66_OPEN_LED
- J7 pad 4: unconnected-(J7-Pad4) -> /U2/ZC66_CLOSE_LED
- J7 pad 5: unconnected-(J7-Pad5) -> /U2/ZC64_CLOSE_MOTOR
- J7 pad 6: unconnected-(J7-Pad6) -> /U2/ZC64_OPEN_MOTOR
- J8 pad 1: unconnected-(J8-Pad1) -> /U3 - U4/ZC67_CLOSE_LED
- J8 pad 2: unconnected-(J8-Pad2) -> /U3 - U4/ZC67_OPEN_LED
- J8 pad 3: unconnected-(J8-Pad3) -> /U3 - U4/ZC66_CLOSE_MOTOR
- J8 pad 4: unconnected-(J8-Pad4) -> /U3 - U4/ZC66_OPEN_MOTOR
- J8 pad 5: unconnected-(J8-Pad5) -> /U3 - U4/ZC65_CLOSE_MOTOR
- J8 pad 6: unconnected-(J8-Pad6) -> /U3 - U4/ZC65_OPEN_MOTOR
- J9 pad 1: unconnected-(J9-Pad1) -> /U3 - U4/ZC68_OPEN_MOTOR
- J9 pad 2: unconnected-(J9-Pad2) -> /U3 - U4/ZC68_CLOSE_MOTOR
- J9 pad 3: unconnected-(J9-Pad3) -> /U3 - U4/ZC67_OPEN_MOTOR
- J9 pad 4: unconnected-(J9-Pad4) -> /U3 - U4/ZC67_CLOSE_MOTOR
- J9 pad 5: unconnected-(J9-Pad5) -> /U3 - U4/ZC68_OPEN_LED
- J9 pad 6: unconnected-(J9-Pad6) -> /U3 - U4/ZC68_CLOSE_LED
- U3 pad 1: /U3 - U4/U3-GPB0 -> U3-GPB0
- U3 pad 2: /U3 - U4/U3-GPB1 -> U3-GPB1
- U3 pad 3: /U3 - U4/U3-GPB2 -> U3-GPB2
- U3 pad 4: /U3 - U4/U3-GPB3 -> U3-GPB3
- U3 pad 5: U3-GPB4 -> /U3 - U4/U3-GPB4
- U3 pad 6: U3-GPB5 -> /U3 - U4/U3-GPB5
- U3 pad 7: U3-GPB6 -> /U3 - U4/U3-GPB6
- U3 pad 8: U3-GPB7 -> /U3 - U4/U3-GPB7
Routing:
- net /U2/ZC66_CLOSE_LED: track 0.00 -> 54.0 mm
- net /U2/ZC66_OPEN_LED: track 0.00 -> 47.8 mm
- net /U2/U2-GPA0: track 0.00 -> 47.4 mm
- net /U2/ZC62_CLOSE_LED: track 0.00 -> 47.2 mm
- net ZC61_OPEN_LED: track 0.00 -> 45.7 mm
- net /U2/U2-GPA1: track 0.00 -> 43.7 mm
- net /U2/ZC62_OPEN_LED: track 0.00 -> 43.2 mm
- net /U2/ZC65_CLOSE_LED: track 0.00 -> 39.8 mm
- net /U2/U2-GPA2: track 0.00 -> 39.7 mm
- net /U3 - U4/U3-GPB7: track 0.00 -> 39.4 mm
- net +3V3: track 91.2 -> 52.5 mm
- net /U2/U2-GPA3: track 0.00 -> 35.4 mm
- net /U3 - U4/U3-GPB6: track 0.00 -> 34.8 mm
- net /U2/ZC65_OPEN_LED: track 0.00 -> 34.5 mm
- net /U3 - U4/U3-GPB5: track 0.00 -> 31.6 mm
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- removed copper zone on F.Cu, net +3V3

Commit message: Ekspander U5 - U6 update
Parts:
- added C21: 0.1uF, Capacitor_SMD:C_0805_2012Metric_Pad1.18x1.45mm_HandSolder, F.Cu at (195.5, 47.8)
- added C22: 0.1uF, Capacitor_SMD:C_0805_2012Metric_Pad1.18x1.45mm_HandSolder, F.Cu at (226.0, 47.7)
- added C23: 0.1uF, Capacitor_SMD:C_0805_2012Metric_Pad1.18x1.45mm_HandSolder, F.Cu at (256.9, 48.3)
- added C24: 0.1uF, Capacitor_SMD:C_0805_2012Metric_Pad1.18x1.45mm_HandSolder, F.Cu at (287.9, 48.5)
- added C25: 0.1uF, Capacitor_SMD:C_0805_2012Metric_Pad1.18x1.45mm_HandSolder, F.Cu at (316.4, 48.3)
- added C26: 0.1uF, Capacitor_SMD:C_0805_2012Metric_Pad1.18x1.45mm_HandSolder, F.Cu at (345.1, 48.3)
- added U23: ITS716G, Package_SO:SOIC-20W_7.5x12.8mm_P1.27mm, F.Cu at (201.1, 40.5)
- added U24: ITS716G, Package_SO:SOIC-20W_7.5x12.8mm_P1.27mm, F.Cu at (231.7, 40.5)
- added U25: LTV-847, Package_DIP:DIP-16_W7.62mm, F.Cu at (212.1, 35.6)
- added U26: LTV-847, Package_DIP:DIP-16_W7.62mm, F.Cu at (244.3, 35.4)
- added U27: ITS716G, Package_SO:SOIC-20W_7.5x12.8mm_P1.27mm, F.Cu at (262.6, 40.4)
- added U28: ITS716G, Package_SO:SOIC-20W_7.5x12.8mm_P1.27mm, F.Cu at (293.6, 40.5)
- added U29: LTV-847, Package_DIP:DIP-16_W7.62mm, F.Cu at (274.4, 35.5)
- added U30: LTV-847, Package_DIP:DIP-16_W7.62mm, F.Cu at (303.9, 35.5)
- added U31: ITS716G, Package_SO:SOIC-20W_7.5x12.8mm_P1.27mm, F.Cu at (322.1, 40.5)
- added U32: ITS716G, Package_SO:SOIC-20W_7.5x12.8mm_P1.27mm, F.Cu at (350.8, 40.4)
- added U33: LTV-847, Package_DIP:DIP-16_W7.62mm, F.Cu at (333.1, 36.4)
- moved U4 33.0 mm to (209.1, 58.9)
- moved U7 26.6 mm to (372.0, 61.9)
- moved C10 26.1 mm to (38.4, 74.0), turned to -90 degrees
- moved U8 25.2 mm to (418.8, 62.0)
- moved U6 20.2 mm to (319.8, 54.2)
- moved U5 17.3 mm to (261.6, 53.3)
- moved U20 8.98 mm to (193.1, 54.1)
- moved C17 0.45 mm to (86.7, 47.7)
Connections:
- J10 pad 1: unconnected-(J10-Pad1) -> /U3 - U4/ZC69_CLOSE_MOTOR
- J10 pad 2: unconnected-(J10-Pad2) -> /U3 - U4/ZC69_OPEN_MOTOR
- J10 pad 3: unconnected-(J10-Pad3) -> /U3 - U4/ZC69_CLOSE_LED
- J10 pad 4: unconnected-(J10-Pad4) -> /U3 - U4/ZC69_OPEN_LED
- J10 pad 5: unconnected-(J10-Pad5) -> /U3 - U4/ZC70_CLOSE_LED
- J10 pad 6: unconnected-(J10-Pad6) -> /U3 - U4/ZC70_OPEN_LED
- J11 pad 1: unconnected-(J11-Pad1) -> /U3 - U4/ZC72_OPEN_LED
- J11 pad 2: unconnected-(J11-Pad2) -> /U3 - U4/ZC72_CLOSE_LED
- J11 pad 3: unconnected-(J11-Pad3) -> /U3 - U4/ZC71_OPEN_LED
- J11 pad 4: unconnected-(J11-Pad4) -> /U3 - U4/ZC71_CLOSE_LED
- J11 pad 5: unconnected-(J11-Pad5) -> /U3 - U4/ZC70_CLOSE_MOTOR
- J11 pad 6: unconnected-(J11-Pad6) -> /U3 - U4/ZC70_OPEN_MOTOR
- J12 pad 1: unconnected-(J12-Pad1) -> ZC74_CLOSE_LED
- J12 pad 2: unconnected-(J12-Pad2) -> ZC74_OPEN_LED
- J12 pad 3: unconnected-(J12-Pad3) -> ZC72_CLOSE_MOTOR
- J12 pad 4: unconnected-(J12-Pad4) -> ZC72_OPEN_MOTOR
- J12 pad 5: unconnected-(J12-Pad5) -> ZC71_CLOSE_MOTOR
- J12 pad 6: unconnected-(J12-Pad6) -> ZC71_OPEN_MOTOR
- J13 pad 1: unconnected-(J13-Pad1) -> /U5/ZC74_CLOSE_MOTOR
- J13 pad 2: unconnected-(J13-Pad2) -> /U5/ZC74_OPEN_MOTOR
- J13 pad 3: unconnected-(J13-Pad3) -> /U5/ZC73_CLOSE_MOTOR
- J13 pad 4: unconnected-(J13-Pad4) -> /U5/ZC73_OPEN_MOTOR
- J13 pad 5: unconnected-(J13-Pad5) -> ZC73_CLOSE_LED
- J13 pad 6: unconnected-(J13-Pad6) -> ZC73_OPEN_LED
- J14 pad 1: unconnected-(J14-Pad1) -> /U5/ZC75_OPEN_MOTOR
- J14 pad 2: unconnected-(J14-Pad2) -> /U5/ZC75_CLOSE_MOTOR
- J14 pad 3: unconnected-(J14-Pad3) -> ZC76_OPEN_LED
- J14 pad 4: unconnected-(J14-Pad4) -> ZC76_CLOSE_LED
- J14 pad 5: unconnected-(J14-Pad5) -> ZC75_CLOSE_LED
- J14 pad 6: unconnected-(J14-Pad6) -> ZC75_OPEN_LED
- J15 pad 1: unconnected-(J15-Pad1) -> ZC78_CLOSE_LED
- J15 pad 2: unconnected-(J15-Pad2) -> ZC78_OPEN_LED
- J15 pad 3: unconnected-(J15-Pad3) -> ZC77_CLOSE_LED
- J15 pad 4: unconnected-(J15-Pad4) -> ZC77_OPEN_LED
- J15 pad 5: unconnected-(J15-Pad5) -> ZC76_CLOSE_MOTOR
- J15 pad 6: unconnected-(J15-Pad6) -> ZC76_OPEN_MOTOR
- J16 pad 1: unconnected-(J16-Pad1) -> ZC79_CLOSE_LED
- J16 pad 2: unconnected-(J16-Pad2) -> ZC79_OPEN_LED
- J16 pad 3: unconnected-(J16-Pad3) -> /U6/ZC78_CLOSE_MOTOR
- J16 pad 4: unconnected-(J16-Pad4) -> /U6/ZC78_OPEN_MOTOR
- J16 pad 5: unconnected-(J16-Pad5) -> /U6/ZC77_CLOSE_MOTOR
- J16 pad 6: unconnected-(J16-Pad6) -> /U6/ZC77_OPEN_MOTOR
- J17 pad 1: unconnected-(J17-Pad1) -> /U6/ZC80_CLOSE_MOTOR
- J17 pad 2: unconnected-(J17-Pad2) -> /U6/ZC80_OPEN_MOTOR
- J17 pad 3: unconnected-(J17-Pad3) -> /U6/ZC79_CLOSE_MOTOR
- J17 pad 4: unconnected-(J17-Pad4) -> /U6/ZC79_OPEN_MOTOR
- J17 pad 5: unconnected-(J17-Pad5) -> ZC80_OPEN_LED
- J17 pad 6: unconnected-(J17-Pad6) -> ZC80_CLOSE_LED
- U19 pad 10: /U3 - U4/U3-GPA4 -> /U3 - U4/U3-GPA0
- U19 pad 12: /U3 - U4/U3-GPA5 -> /U3 - U4/U3-GPA1
- U19 pad 14: /U3 - U4/U3-GPA6 -> /U3 - U4/U3-GPA2
- U19 pad 16: /U3 - U4/U3-GPA7 -> /U3 - U4/U3-GPA3
- U20 pad 10: unconnected-(U20-Pad10) -> /U3 - U4/U4-GPB3
- U20 pad 12: unconnected-(U20-Pad12) -> /U3 - U4/U4-GPB2
- U20 pad 14: unconnected-(U20-Pad14) -> /U3 - U4/U4-GPB1
- U20 pad 16: unconnected-(U20-Pad16) -> /U3 - U4/U4-GPB0
- U22 pad 3: /U3 - U4/U2-GPA3 -> /U3 - U4/U3-GPA4
- U22 pad 5: /U3 - U4/U2-GPA2 -> /U3 - U4/U3-GPA5
- U22 pad 7: /U3 - U4/U2-GPA1 -> /U3 - U4/U3-GPA6
- U22 pad 9: /U3 - U4/U2-GPA0 -> /U3 - U4/U3-GPA7
Routing:
- net /U3 - U4/ZC70_OPEN_LED: track 0.00 -> 53.9 mm
- net /U3 - U4/U4-GPA0: track 0.00 -> 44.9 mm
- net /U3 - U4/ZC69_OPEN_LED: track 0.00 -> 43.5 mm
- net /U6/U6-GPA4: track 0.00 -> 43.4 mm
- net /U5/U5-GPA4: track 0.00 -> 39.4 mm
- net /U3 - U4/ZC70_CLOSE_LED: track 0.00 -> 38.8 mm
- net ZC78_OPEN_LED: track 0.00 -> 38.3 mm
- net /U6/U6-GPA5: track 0.00 -> 37.9 mm
- net /U3 - U4/U4-GPA1: track 0.00 -> 36.3 mm
- net /U3 - U4/U4-GPB7: track 0.00 -> 36.2 mm
- net /U5/U5-GPA5: track 0.00 -> 36.1 mm
- net /U6/U6-GPA3: track 0.00 -> 35.9 mm
- net /U3 - U4/U3-GPA3: track 0.00 -> 35.1 mm
- net /U6/U6-GPA6: track 0.00 -> 35.1 mm
- net ZC74_OPEN_LED: track 0.00 -> 34.2 mm
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- added copper zone on B.Cu, net +24V

Commit message: Ekspander 24V update
Parts:
- added C27: 0.1uF, Capacitor_SMD:C_0805_2012Metric_Pad1.18x1.45mm_HandSolder, F.Cu at (372.6, 48.2)
- added C28: 0.1uF, Capacitor_SMD:C_0805_2012Metric_Pad1.18x1.45mm_HandSolder, F.Cu at (400.3, 48.4)
- added C29: 0.1uF, Capacitor_SMD:C_0805_2012Metric_Pad1.18x1.45mm_HandSolder, F.Cu at (428.5, 48.5)
- added C30: 0.1uF, Capacitor_SMD:C_0805_2012Metric_Pad1.18x1.45mm_HandSolder, F.Cu at (456.8, 48.8)
- added C31: 0.1uF, Capacitor_SMD:C_0805_2012Metric_Pad1.18x1.45mm_HandSolder, F.Cu at (38.9, 73.8)
- added J22: DG127A-5.08-06P-14-00AH, 1_tme:DG127A50806P1400AH, F.Cu at (446.8, 18.1)
- added J23: DG127A-5.08-06P-14-00AH, 1_tme:DG127A50806P1400AH, F.Cu at (468.2, 18.1)
- added R2: 10K, PCM_Resistor_SMD_AKL:R_0805_2012Metric_Pad1.20x1.40mm_HandSolder, F.Cu at (51.9, 76.3)
- added R3: 10K, PCM_Resistor_SMD_AKL:R_0805_2012Metric_Pad1.20x1.40mm_HandSolder, F.Cu at (106.8, 77.1)
- added R4: 10K, PCM_Resistor_SMD_AKL:R_0805_2012Metric_Pad1.20x1.40mm_HandSolder, F.Cu at (183.0, 80.1)
- added R5: 10K, PCM_Resistor_SMD_AKL:R_0805_2012Metric_Pad1.20x1.40mm_HandSolder, F.Cu at (219.4, 83.0)
- added R6: 10K, PCM_Resistor_SMD_AKL:R_0805_2012Metric_Pad1.20x1.40mm_HandSolder, F.Cu at (272.0, 77.5)
- added R7: 10K, PCM_Resistor_SMD_AKL:R_0805_2012Metric_Pad1.20x1.40mm_HandSolder, F.Cu at (351.1, 81.0)
- added R8: 10K, PCM_Resistor_SMD_AKL:R_0805_2012Metric_Pad1.20x1.40mm_HandSolder, F.Cu at (344.2, 71.0)
- added R9: 10K, PCM_Resistor_SMD_AKL:R_0805_2012Metric_Pad1.20x1.40mm_HandSolder, F.Cu at (344.2, 74.0)
- added U34: LTV-847, Package_DIP:DIP-16_W7.62mm, F.Cu at (360.8, 36.0)
- added U35: ITS716G, Package_SO:SOIC-20W_7.5x12.8mm_P1.27mm, F.Cu at (378.2, 40.4)
- added U36: ITS716G, Package_SO:SOIC-20W_7.5x12.8mm_P1.27mm, F.Cu at (406.1, 40.4)
- added U37: LTV-847, Package_DIP:DIP-16_W7.62mm, F.Cu at (387.9, 36.0)
- added U38: ITS716G, Package_SO:SOIC-20W_7.5x12.8mm_P1.27mm, F.Cu at (434.2, 40.5)
- added U39: ITS716G, Package_SO:SOIC-20W_7.5x12.8mm_P1.27mm, F.Cu at (462.5, 40.8)
- added U40: LTV-847, Package_DIP:DIP-16_W7.62mm, F.Cu at (416.1, 36.1)
- added U41: LTV-847, Package_DIP:DIP-16_W7.62mm, F.Cu at (444.2, 36.1)
- C1, C2: value 100nF -> 0.1uF; footprint Capacitor_THT:C_Disc_D3.0mm_W2.0mm_P2.50mm -> Capacitor_SMD:C_0805_2012Metric_Pad1.18x1.45mm_HandSolder
- moved C16 358.4 mm to (427.9, 76.8), turned to -90 degrees
- moved C15 303.0 mm to (372.4, 75.5), turned to -90 degrees
- moved C14 248.2 mm to (317.1, 75.8), turned to -90 degrees
- moved J1 216.9 mm to (489.6, 18.1)
- moved C13 189.9 mm to (258.9, 74.9), turned to -90 degrees
- moved C12 137.0 mm to (206.4, 80.5), turned to -90 degrees
- moved C11 100.4 mm to (169.9, 77.4), turned to -90 degrees
- moved C10 55.7 mm to (94.0, 74.5)
- moved U8 13.6 mm to (430.5, 55.1)
- moved U7 8.69 mm to (375.1, 53.8)
- moved C2 3.85 mm to (62.6, 48.3), turned to 0 degrees
- moved C1 1.79 mm to (22.4, 48.6)
Connections:
- IC1 pad 15: unconnected-(IC1-IO3-Pad15) -> RESET_U8
- IC1 pad 16: unconnected-(IC1-IO46-Pad16) -> RESET_U7
- IC1 pad 17: unconnected-(IC1-IO9-Pad17) -> RESET_U6
- IC1 pad 18: unconnected-(IC1-IO10-Pad18) -> RESET_U5
- IC1 pad 19: unconnected-(IC1-IO11-Pad19) -> RESET_U4
- IC1 pad 20: unconnected-(IC1-IO12-Pad20) -> RESET_U3
- IC1 pad 21: unconnected-(IC1-IO13-Pad21) -> RESET_U2
- IC1 pad 22: unconnected-(IC1-IO14-Pad22) -> RESET_U1
- IC1 pad 38: unconnected-(IC1-IO2-Pad38) -> SCK
- IC1 pad 39: unconnected-(IC1-IO1-Pad39) -> SDA
- IC1 pad 4: SDA -> unconnected-(IC1-IO4-Pad4)
- IC1 pad 5: SCK -> unconnected-(IC1-IO5-Pad5)
- J1 pad 3: unconnected-(J1-Pad3) -> GND
- J1 pad 4: unconnected-(J1-Pad4) -> GND
- J1 pad 5: SDA -> GND
- J1 pad 6: SCK -> GND
- J18 pad 1: unconnected-(J18-Pad1) -> /U7 - U8/ZC81_CLOSE_MOTOR
- J18 pad 2: unconnected-(J18-Pad2) -> /U7 - U8/ZC81_OPEN_MOTOR
- J18 pad 3: unconnected-(J18-Pad3) -> ZCX01_OPEN_LED
- J18 pad 4: unconnected-(J18-Pad4) -> ZCX01_CLOSE_LED
- J18 pad 5: unconnected-(J18-Pad5) -> ZC81_CLOSE_LED
- J18 pad 6: unconnected-(J18-Pad6) -> ZC81_OPEN_LED
- J19 pad 1: unconnected-(J19-Pad1) -> ZCX03_OPEN_LED
- J19 pad 2: unconnected-(J19-Pad2) -> ZCX03_CLOSE_LED
- J19 pad 3: unconnected-(J19-Pad3) -> ZCX02_CLOSE_LED
- J19 pad 4: unconnected-(J19-Pad4) -> ZCX02_OPEN_LED
- J19 pad 5: unconnected-(J19-Pad5) -> /U7 - U8/ZCX01_CLOSE_MOTOR
- J19 pad 6: unconnected-(J19-Pad6) -> /U7 - U8/ZCX01_OPEN_MOTOR
- J20 pad 1: unconnected-(J20-Pad1) -> ZCX04_CLOSE_LED
- J20 pad 2: unconnected-(J20-Pad2) -> ZCX04_OPEN_LED
- J20 pad 3: unconnected-(J20-Pad3) -> /U7 - U8/ZCX03_CLOSE_MOTOR
- J20 pad 4: unconnected-(J20-Pad4) -> /U7 - U8/ZCX03_OPEN_MOTOR
- J20 pad 5: unconnected-(J20-Pad5) -> /U7 - U8/ZCX02_CLOSE_MOTOR
- J20 pad 6: unconnected-(J20-Pad6) -> /U7 - U8/ZCX02_OPEN_MOTOR
- J21 pad 1: unconnected-(J21-Pad1) -> /U7 - U8/ZCX05_CLOSE_MOTOR
- J21 pad 2: unconnected-(J21-Pad2) -> /U7 - U8/ZCX05_OPEN_MOTOR
- J21 pad 3: unconnected-(J21-Pad3) -> /U7 - U8/ZCX04_CLOSE_MOTOR
- J21 pad 4: unconnected-(J21-Pad4) -> /U7 - U8/ZCX04_OPEN_MOTOR
- J21 pad 5: unconnected-(J21-Pad5) -> ZCX05_OPEN_LED
- J21 pad 6: unconnected-(J21-Pad6) -> ZCX05_CLOSE_LED
- U1 pad 18: unconnected-(U1-~{RESET}-Pad18) -> RESET_U1
- U2 pad 18: unconnected-(U2-~{RESET}-Pad18) -> RESET_U2
- U3 pad 18: unconnected-(U3-~{RESET}-Pad18) -> RESET_U3
- U4 pad 18: unconnected-(U4-~{RESET}-Pad18) -> RESET_U4
- U5 pad 12: /U5/SCK -> SCK
- U5 pad 13: /U5/SDA -> SDA
- U5 pad 18: unconnected-(U5-~{RESET}-Pad18) -> RESET_U5
- U6 pad 18: unconnected-(U6-~{RESET}-Pad18) -> RESET_U6
- U7 pad 18: unconnected-(U7-~{RESET}-Pad18) -> RESET_U7
- U8 pad 18: unconnected-(U8-~{RESET}-Pad18) -> RESET_U8
Routing:
- net +3V3: track 52.5 -> 676.5 mm, vias 0 -> 2
- net SCK: track 0.00 -> 449.9 mm, vias 0 -> 1
- net SDA: track 0.00 -> 443.3 mm, vias 0 -> 1
- net +24V: track 16.5 -> 308.6 mm, vias 4 -> 140
- net RESET_U1: track 0.00 -> 193.8 mm, vias 0 -> 2
- net RESET_U2: track 0.00 -> 139.4 mm, vias 0 -> 2
- net RESET_U3: track 0.00 -> 57.1 mm, vias 0 -> 2
- net /U7 - U8/U8-GPA4: track 0.00 -> 40.7 mm
- net /U7 - U8/U7-GPA4: track 0.00 -> 40.7 mm
- net /U7 - U8/U7-GPA5: track 0.00 -> 37.1 mm
- net /U7 - U8/U8-GPA5: track 0.00 -> 37.0 mm
- net RESET_U4: track 0.00 -> 35.8 mm
- net /U7 - U8/U8-GPA3: track 0.00 -> 34.9 mm
- net /U7 - U8/U8-GPA6: track 0.00 -> 33.7 mm
- net /U7 - U8/U7-GPA3: track 0.00 -> 33.3 mm
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
Commit message: Ekspander 100x - PCB layout V1
Routing:
- net +24V: vias 140 -> 182
- added copper zone on In1.Cu, net +24V
- added copper zone on In2.Cu, net +24V
Other:
- board text added: "10,5A"
- board text added: "14A"
- board text added: "17,5A"
- board text added: "21A"
- board text added: "24,5A"
- board text added: "28A"
- board text added: "3,5A"
- board text added: "31,5A"
- board text added: "35A"
- board text added: "38,5A"
- board text added: "42A"
- board text added: "45,5A"
- board text added: "49A"
- board text added: "52,5A"
- board text added: "7A"

Commit message: Ekspander 100x - PCB layout V2
Parts:
- moved U8 358.5 mm to (73.3, 85.8)
- moved C16 319.3 mm to (110.3, 109.8), turned to 0 degrees
- moved U7 318.2 mm to (58.3, 83.8)
- moved U41 311.3 mm to (136.3, 81.8)
- moved U37 307.2 mm to (84.3, 82.8)
- moved R8 279.4 mm to (69.3, 120.8)
- moved C15 264.0 mm to (110.3, 106.8), turned to 0 degrees
- moved R9 254.9 mm to (93.3, 118.8)
- moved R6 244.8 mm to (29.3, 109.8), turned to 0 degrees
- moved R7 241.5 mm to (110.3, 99.8)
- moved J1 236.4 mm to (253.3, 18.1)
- moved C14 207.0 mm to (115.3, 121.8), turned to 0 degrees
- moved U6 206.9 mm to (114.3, 78.8)
- moved U34 206.6 mm to (158.3, 76.8)
- moved J23 193.5 mm to (274.7, 18.1)
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Connections:
- J1 pad 2: GND -> +24V
- J1 pad 3: GND -> +24V
- J23 pad 1: /U7 - U8/ZCX07_OPEN_MOTOR -> GND
- J23 pad 2: /U7 - U8/ZCX07_CLOSE_MOTOR -> GND
- J23 pad 3: +24V -> GND
- U12 pad 13: /ZC60_OPEN_MOTOR -> /ZC60_CLOSE_MOTOR
- U12 pad 14: /ZC60_CLOSE_MOTOR -> /ZC60_OPEN_MOTOR
- U12 pad 17: /ZC59_OPEN_MOTOR -> /ZC59_CLOSE_MOTOR
- U12 pad 18: /ZC59_CLOSE_MOTOR -> /ZC59_OPEN_MOTOR
- U16 pad 13: /U2/ZC64_OPEN_MOTOR -> /U2/ZC64_CLOSE_MOTOR
- U16 pad 14: /U2/ZC64_CLOSE_MOTOR -> /U2/ZC64_OPEN_MOTOR
Routing:
- net +3V3: track 676.5 -> 52.5 mm, vias 2 -> 0
- net SCK: track 449.9 -> 0.00 mm, vias 1 -> 0
- net SDA: track 443.3 -> 0.00 mm, vias 1 -> 0
- net GND: track 55.0 -> 388.1 mm, vias 339 -> 74
- net +24V: track 308.6 -> 95.0 mm, vias 182 -> 32
- net RESET_U1: track 193.8 -> 0.00 mm, vias 2 -> 0
- net RESET_U2: track 139.4 -> 0.00 mm, vias 2 -> 0
- net /ZC58_CLOSE_LED: track 58.4 -> 0.00 mm
- net RESET_U3: track 57.1 -> 0.00 mm, vias 2 -> 0
- net /ZC57_OPEN_LED: track 55.6 -> 0.00 mm
- net /U2/ZC66_CLOSE_LED: track 54.0 -> 0.00 mm
- net /U3 - U4/ZC70_OPEN_LED: track 53.9 -> 0.00 mm
- net /U2/ZC66_OPEN_LED: track 47.8 -> 0.00 mm
- net /U2/U2-GPA0: track 47.4 -> 0.00 mm
- net /U2/ZC62_CLOSE_LED: track 47.2 -> 0.00 mm
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- added copper zone on In1.Cu, net GND
- added copper zone on In2.Cu, net GND
Other:
- board text removed: "10,5A"
- board text removed: "14A"
- board text removed: "17,5A"
- board text removed: "21A"
- board text removed: "24,5A"
- board text removed: "28A"
- board text removed: "3,5A"
- board text removed: "31,5A"
- board text removed: "35A"
- board text removed: "38,5A"
- board text removed: "42A"
- board text removed: "45,5A"
- board text removed: "49A"
- board text removed: "52,5A"
- board text removed: "7A"
