File: pcb/ekspander_100x_i2c/ekspander_100x_i2c.kicad_pcb (KiCad board)
At the start: 4 copper layers, 500 x 108.8 mm, 282 parts, among them IC1 ESP32-S3-WROOM-1U-N16R8, J1 DG127A-5.08-06P-14-00AH, J10 DG127A-5.08-06P-14-00AH, J11 DG127A-5.08-06P-14-00AH, J12 DG127A-5.08-06P-14-00AH, J13 DG127A-5.08-06P-14-00AH, J14 DG127A-5.08-06P-14-00AH, J15 DG127A-5.08-06P-14-00AH, J16 DG127A-5.08-06P-14-00AH, J17 DG127A-5.08-06P-14-00AH, J18 DG127A-5.08-06P-14-00AH, J19 DG127A-5.08-06P-14-00AH, J2 DG127A-5.08-06P-14-00AH, J20 DG127A-5.08-06P-14-00AH, J21 DG127A-5.08-06P-14-00AH, J22 DG127A-5.08-06P-14-00AH, J23 DG127A-5.08-06P-14-00AH, J25 USB4145-03-0230-C, J3 DG127A-5.08-06P-14-00AH, J4 DG127A-5.08-06P-14-00AH, J5 DG127A-5.08-06P-14-00AH, J6 DG127A-5.08-06P-14-00AH, J7 DG127A-5.08-06P-14-00AH, J8 DG127A-5.08-06P-14-00AH, J9 DG127A-5.08-06P-14-00AH, K1 G5Q-1A, K10 G5Q-1A, K11 G5Q-1A, K12 G5Q-1A, K13 G5Q-1A, K14 G5Q-1A, K15 G5Q-1A, K16 G5Q-1A, K17 G5Q-1A, K18 G5Q-1A, K19 G5Q-1A, K2 G5Q-1A, K20 G5Q-1A, K21 G5Q-1A, K22 G5Q-1A, K23 G5Q-1A, K24 G5Q-1A, K25 G5Q-1A, K26 G5Q-1A, K27 G5Q-1A, K28 G5Q-1A, K29 G5Q-1A, K3 G5Q-1A, K30 G5Q-1A, K31 G5Q-1A, K32 G5Q-1A, K33 G5Q-1A, K34 G5Q-1A, K35 G5Q-1A, K36 G5Q-1A, K37 G5Q-1A, K38 G5Q-1A, K39 G5Q-1A, K4 G5Q-1A, K40 G5Q-1A, K41 G5Q-1A, K42 G5Q-1A, K43 G5Q-1A, K44 G5Q-1A, K45 G5Q-1A, K46 G5Q-1A, K47 G5Q-1A, K48 G5Q-1A, K49 G5Q-1A, K5 G5Q-1A, K50 G5Q-1A, K6 G5Q-1A, K7 G5Q-1A, K8 G5Q-1A, K9 G5Q-1A, U1 MCP23017_SP, U10 ITS716G, U11 LTV-847, U12 ITS716G, U13 AP63203WU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

Commit message: Ekspander 100x - RS485
Parts:
- added C34: 0.1uF, Capacitor_SMD:C_0805_2012Metric_Pad1.18x1.45mm_HandSolder, F.Cu at (321.2, 95.8)
- added U42: MAX3485, Package_SO:SOIC-8_3.9x4.9mm_P1.27mm, F.Cu at (315.2, 98.2)
Connections:
- IC1 pad 10: unconnected-(IC1-IO17-Pad10) -> /esp32/RX_TX1
- IC1 pad 11: unconnected-(IC1-IO18-Pad11) -> /esp32/TX_RX1
- IC1 pad 12: unconnected-(IC1-IO8-Pad12) -> /esp32/RE/DE
- J22 pad 1: ZCX06_OPEN_LED -> unconnected-(J22-Pad1)
- J22 pad 2: ZCX06_CLOSE_LED -> unconnected-(J22-Pad2)
- J22 pad 3: ZCX07_CLOSE_LED -> unconnected-(J22-Pad3)
- J22 pad 4: ZCX07_OPEN_LED -> unconnected-(J22-Pad4)
- J22 pad 5: /U7 - U8/ZCX06_OPEN_MOTOR -> RS485/A
- J22 pad 6: /U7 - U8/ZCX06_CLOSE_MOTOR -> RS485/B
Routing:
- net RS485/A: track 0.00 -> 269.7 mm
- net RS485/B: track 0.00 -> 255.8 mm
- net /esp32/RE/DE: track 0.00 -> 65.1 mm, vias 0 -> 2
- net /esp32/RX_TX1: track 0.00 -> 63.7 mm, vias 0 -> 2
- net /esp32/TX_RX1: track 0.00 -> 61.2 mm, vias 0 -> 2
- net +3V3: track 258.8 -> 281.2 mm
- net GND: track 499.2 -> 509.5 mm, vias 99 -> 100

Commit message: Ekspander 100x - RESET - BOOT - switches
Parts:
- added C35: 0.1uF, Capacitor_SMD:C_0805_2012Metric_Pad1.18x1.45mm_HandSolder, F.Cu at (234.8, 82.8)
- added R75: 10K, PCM_Resistor_SMD_AKL:R_0805_2012Metric_Pad1.20x1.40mm_HandSolder, F.Cu at (231.8, 86.8)
- added S1: 1301.9315, 1_tme:13019319, F.Cu at (344.1, 88.0)
- added S2: 1301.9315, 1_tme:13019319, F.Cu at (344.1, 97.1)
- moved R16 7.08 mm to (226.5, 92.2), turned to -90 degrees
Connections:
- IC1 pad 16: RESET_U7 -> unconnected-(IC1-IO46-Pad16)
- IC1 pad 23: unconnected-(IC1-IO21-Pad23) -> RESET_U7
- IC1 pad 27: unconnected-(IC1-IO0-Pad27) -> Net-(IC1-IO0)
Routing:
- net Net-(IC1-EN): track 11.0 -> 146.3 mm, vias 0 -> 2
- net Net-(IC1-IO0): track 0.00 -> 131.2 mm, vias 0 -> 6
- net GND: track 509.5 -> 533.3 mm
- net RESET_U1: track 202.0 -> 207.1 mm, vias 0 -> 2
- net RESET_U7: track 212.2 -> 216.9 mm
- net SCK: track 473.8 -> 477.1 mm
- net +3V3: track 281.2 -> 280.2 mm
