File: pcb/ekspander_100x_i2c/_autosave-esp32.kicad_sch (KiCad schematic)
At the start: 32 parts, among them IC1 ESP32-S3-WROOM-1U-N16R8, J25 USB4145-03-0230-C, U13 AP63203WU, U39 USBLC6-2SC6, U41 CP2102N-A02-GQFN20

Commit message: Ekspander 100x - LEDs
Changed lines of the file:
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@@
 	)
 	(junction
+		(at 86.36 71.12)
+		(diameter 0)
+		(color 0 0 0 0)
+	)
+	(junction
 		(at 76.2 102.87)
 		(diameter 0)
@@
 		(color 0 0 0 0)
 	)
-	(junction
-		(at 87.63 71.12)
-		(diameter 0)
-		(color 0 0 0 0)
-	)
 	(no_connect
 		(at 236.22 93.98)
@@
 	(wire
 		(pts
+			(xy 86.36 71.12) (xy 90.17 71.12)
+		)
+		(stroke
+			(width 0)
+			(type default)
+		)
+	)
+	(wire
+		(pts
 			(xy 34.29 21.59) (xy 34.29 25.4)
 		)
@@
 	(wire
 		(pts
-			(xy 82.55 71.12) (xy 87.63 71.12)
+			(xy 82.55 71.12) (xy 86.36 71.12)
 		)
 		(stroke
@@
 	(wire
 		(pts
-			(xy 87.63 71.12) (xy 90.17 71.12)
-		)
-		(stroke
-			(width 0)
-			(type default)
-		)
-	)
-	(wire
-		(pts
 			(xy 172.72 53.34) (xy 172.72 60.96)
 		)
@@
 	(wire
 		(pts
-			(xy 87.63 71.12) (xy 87.63 67.31)
+			(xy 86.36 71.12) (xy 86.36 67.31)
 		)
 		(stroke
@@
 	(symbol
 		(lib_id "power:+5VD")
-		(at 87.63 67.31 0)
+		(at 86.36 67.31 0)
 		(unit 1)
 		(exclude_from_sim no)
@@
 		(dnp no)
 		(property "Reference" "#PWR0113"
-			(at 87.63 71.12 0)
+			(at 86.36 71.12 0)
 			(effects
 				(font
@@
 		)
 		(property "Value" "+3V3"
-			(at 87.63 63.246 0)
+			(at 86.36 63.246 0)
 			(effects
 				(font
@@
 		)
 		(property "Footprint" ""
-			(at 87.63 67.31 0)
+			(at 86.36 67.31 0)
 			(effects
 				(font
@@
 		)
 		(property "Datasheet" ""
-			(at 87.63 67.31 0)
+			(at 86.36 67.31 0)
 			(effects
 				(font
@@
 		)
 		(property "Description" "Power symbol creates a global label with name \"+5VD\""
-			(at 87.63 67.31 0)
+			(at 86.36 67.31 0)
 			(effects
 				(font
