File: pcb/ekspander_100x_i2c/_autosave-esp32.kicad_sch (KiCad schematic)
At the start: 37 parts, among them IC1 ESP32-S3-WROOM-1U-N16R8, J25 USB4145-03-0230-C, U13 AP63203WU, U39 USBLC6-2SC6, U41 CP2102N-A02-GQFN20, U42 MAX3485

Commit message: Ekspander 100x - RESET - BOOT - switches
Parts:
- added R75: 10K, PCM_Resistor_SMD_AKL:R_0805_2012Metric_Pad1.20x1.40mm_HandSolder, symbol Device:R
Connections:
- net +3V3: now also R75.2
- net GND: now also C35.2
- net at S1.3 (COM_1), S1.4 (COM_2): now also C35.1, IC1.27 (IO0), R75.1; no longer C35.2
Other:
- moved on the sheet: C35
Changed lines of the file:
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@@
 	)
 	(junction
+		(at 78.74 54.61)
+		(diameter 0)
+		(color 0 0 0 0)
+	)
+	(junction
 		(at 82.55 85.09)
 		(diameter 0)
@@
 	)
 	(junction
-		(at 80.01 38.1)
-		(diameter 0)
-		(color 0 0 0 0)
-	)
-	(junction
 		(at 121.92 49.53)
 		(diameter 0)
@@
 	)
 	(junction
+		(at 86.36 68.58)
+		(diameter 0)
+		(color 0 0 0 0)
+	)
+	(junction
 		(at 76.2 107.95)
 		(diameter 0)
@@
 	)
 	(junction
+		(at 88.9 41.91)
+		(diameter 0)
+		(color 0 0 0 0)
+	)
+	(junction
 		(at 76.2 97.79)
 		(diameter 0)
@@
 	)
 	(junction
+		(at 76.2 54.61)
+		(diameter 0)
+		(color 0 0 0 0)
+	)
+	(junction
 		(at 280.67 95.25)
 		(diameter 0)
@@
 		(color 0 0 0 0)
 	)
+	(junction
+		(at 76.2 38.1)
+		(diameter 0)
+		(color 0 0 0 0)
+	)
 	(no_connect
 		(at 236.22 93.98)
@@
 	(wire
 		(pts
+			(xy 86.36 68.58) (xy 78.74 68.58)
+		)
+		(stroke
+			(width 0)
+			(type default)
+		)
+	)
+	(wire
+		(pts
 			(xy 100.33 33.02) (xy 105.41 33.02)
 		)
@@
 	(wire
 		(pts
-			(xy 25.4 53.34) (xy 25.4 57.15)
+			(xy 78.74 54.61) (xy 78.74 57.15)
 		)
 		(stroke
@@
 	(wire
 		(pts
-			(xy 72.39 90.17) (xy 76.2 90.17)
+			(xy 78.74 54.61) (xy 76.2 54.61)
 		)
 		(stroke
@@
 	(wire
 		(pts
-			(xy 242.57 149.86) (xy 243.84 149.86)
+			(xy 25.4 53.34) (xy 25.4 57.15)
 		)
 		(stroke
@@
 	(wire
 		(pts
-			(xy 80.01 38.1) (xy 85.09 38.1)
+			(xy 72.39 90.17) (xy 76.2 90.17)
+		)
+		(stroke
+			(width 0)
+			(type default)
+		)
+	)
+	(wire
+		(pts
+			(xy 242.57 149.86) (xy 243.84 149.86)
 		)
 		(stroke
@@
 	(wire
 		(pts
+			(xy 78.74 68.58) (xy 78.74 64.77)
+		)
+		(stroke
+			(width 0)
+			(type default)
+		)
+	)
+	(wire
+		(pts
 			(xy 260.35 95.25) (xy 261.62 95.25)
 		)
@@
 	(wire
 		(pts
+			(xy 76.2 54.61) (xy 72.39 54.61)
+		)
+		(stroke
+			(width 0)
+			(type default)
+		)
+	)
+	(wire
+		(pts
 			(xy 223.52 55.88) (xy 223.52 54.61)
 		)
@@
 	(wire
 		(pts
+			(xy 76.2 38.1) (xy 85.09 38.1)
+		)
+		(stroke
+			(width 0)
+			(type default)
+		)
+	)
+	(wire
+		(pts
 			(xy 203.2 60.96) (xy 203.2 50.8)
 		)
@@
 	(wire
 		(pts
-			(xy 88.9 30.48) (xy 88.9 44.45)
+			(xy 88.9 30.48) (xy 88.9 41.91)
 		)
 		(stroke
@@
 	(wire
 		(pts
-			(xy 76.2 110.49) (xy 76.2 127)
+			(xy 76.2 38.1) (xy 76.2 54.61)
 		)
 		(stroke
@@
 	(wire
 		(pts
-			(xy 273.05 149.86) (xy 280.67 149.86)
+			(xy 76.2 110.49) (xy 76.2 127)
 		)
 		(stroke
@@
 	(wire
 		(pts
-			(xy 80.01 167.64) (xy 80.01 170.18)
+			(xy 273.05 149.86) (xy 280.67 149.86)
 		)
 		(stroke
@@
 	(wire
 		(pts
-			(xy 260.35 96.52) (xy 260.35 95.25)
+			(xy 80.01 167.64) (xy 80.01 170.18)
 		)
 		(stroke
@@
 	(wire
 		(pts
-			(xy 72.39 54.61) (xy 80.01 54.61)
+			(xy 260.35 96.52) (xy 260.35 95.25)
 		)
 		(stroke
@@
 	(wire
 		(pts
+			(xy 86.36 68.58) (xy 86.36 67.31)
+		)
+		(stroke
+			(width 0)
+			(type default)
+		)
+	)
+	(wire
+		(pts
 			(xy 231.14 149.86) (xy 231.14 151.13)
 		)
@@
 	(wire
 		(pts
+			(xy 80.01 41.91) (xy 88.9 41.91)
+		)
+		(stroke
+			(width 0)
+			(type default)
+		)
+	)
+	(wire
+		(pts
 			(xy 39.37 57.15) (xy 25.4 57.15)
 		)
@@
 	(wire
 		(pts
+			(xy 88.9 41.91) (xy 88.9 44.45)
+		)
+		(stroke
+			(width 0)
+			(type default)
+		)
+	)
+	(wire
+		(pts
 			(xy 72.39 100.33) (xy 76.2 100.33)
 		)
@@
 	(wire
 		(pts
+			(xy 78.74 54.61) (xy 78.74 49.53)
+		)
+		(stroke
+			(width 0)
+			(type default)
+		)
+	)
+	(wire
+		(pts
 			(xy 85.09 17.78) (xy 85.09 30.48)
 		)
@@
 	(wire
 		(pts
-			(xy 80.01 38.1) (xy 54.61 38.1)
+			(xy 54.61 38.1) (xy 76.2 38.1)
 		)
 		(stroke
@@
 	(wire
 		(pts
-			(xy 220.98 31.75) (xy 220.98 43.18)
+			(xy 78.74 49.53) (xy 80.01 49.53)
 		)
 		(stroke
@@
 	(wire
 		(pts
-			(xy 260.35 100.33) (xy 257.81 100.33)
+			(xy 220.98 31.75) (xy 220.98 43.18)
 		)
 		(stroke
@@
 	(wire
 		(pts
-			(xy 33.02 62.23) (xy 39.37 62.23)
+			(xy 260.35 100.33) (xy 257.81 100.33)
 		)
 		(stroke
@@
 	(wire
 		(pts
-			(xy 128.27 63.5) (xy 127 63.5)
+			(xy 33.02 62.23) (xy 39.37 62.23)
 		)
 		(stroke
@@
 	(wire
 		(pts
-			(xy 80.01 46.99) (xy 80.01 38.1)
+			(xy 128.27 63.5) (xy 127 63.5)
 		)
 		(stroke
@@
 	(wire
 		(pts
-			(xy 86.36 71.12) (xy 86.36 67.31)
+			(xy 86.36 71.12) (xy 86.36 68.58)
 		)
 		(stroke
@@
 	(symbol
 		(lib_id "Device:C")
-		(at 80.01 50.8 180)
+		(at 80.01 45.72 180)
 		(unit 1)
 		(exclude_from_sim no)
@@
 		(dnp no)
 		(property "Reference" "C35"
-			(at 78.74 54.356 90)
+			(at 78.74 49.276 90)
 			(effects
 				(font
@@
 		)
 		(property "Value" "0.1uF"
-			(at 81.534 54.864 90)
+			(at 81.534 49.784 90)
 			(effects
 				(font
@@
 		)
 		(property "Footprint" "Capacitor_SMD:C_0805_2012Metric_Pad1.18x1.45mm_HandSolder"
-			(at 79.0448 46.99 0)
+			(at 79.0448 41.91 0)
 			(effects
 				(font
@@
 		)
 		(property "Datasheet" "~"
-			(at 80.01 50.8 0)
+			(at 80.01 45.72 0)
 			(effects
 				(font
@@
 		)
 		(property "Description" "Unpolarized capacitor"
-			(at 80.01 50.8 0)
+			(at 80.01 45.72 0)
 			(effects
 				(font
@@
 					(unit 1)
 				)
+			)
+		)
+	)
+	(symbol
+		(lib_id "Device:R")
+		(at 78.74 60.96 0)
+		(unit 1)
+		(exclude_from_sim no)
+		(in_bom yes)
+		(on_board yes)
+		(dnp no)
+		(fields_autoplaced yes)
+		(property "Reference" "R75"
+			(at 81.28 59.6899 0)
+			(effects
+				(font
+					(size 1.27 1.27)
+				)
+				(justify left)
+			)
+		)
+		(property "Value" "10K"
+			(at 81.28 62.2299 0)
+			(effects
+				(font
+					(size 1.27 1.27)
+				)
+				(justify left)
+			)
+		)
+		(property "Footprint" "PCM_Resistor_SMD_AKL:R_0805_2012Metric_Pad1.20x1.40mm_HandSolder"
+			(at 76.962 60.96 90)
+			(effects
+				(font
+					(size 1.27 1.27)
+				)
+				(hide yes)
+			)
+		)
+		(property "Datasheet" "~"
+			(at 78.74 60.96 0)
+			(effects
+				(font
+					(size 1.27 1.27)
+				)
+				(hide yes)
+			)
+		)
+		(property "Description" "Resistor"
+			(at 78.74 60.96 0)
+			(effects
+				(font
+					(size 1.27 1.27)
+				)
+				(hide yes)
+			)
+		)
+		(property "Cena" "0,04"
+			(at 78.74 60.96 0)
+			(effects
+				(font
+					(size 1.27 1.27)
+				)
+				(hide yes)
+			)
+		)
+		(pin "2"
+		)
+		(pin "1"
+		)
+		(instances
+			(project "ekspander_100x_i2c"
+				(path "/824ceec5-564f-405b-8bea-e5a9f7aa2926/55ba1fbf-ba99-4dff-a5fd-f0299e9a0a1f"
+					(reference "R75")
+					(unit 1)
+				)
