File: mikrokontrolery/esp32/KLP-5e-ESP32-sensor-board/KiCad project/ESP32 sensor board.kicad_pcb (KiCad board)
At the start: 4 copper layers, 89.9 x 52.8 mm, 90 parts, among them J1 USB_C_Receptacle, J2 JST_2mm_LiPo, J3 GSD090012SEU, J4 B4B-XH-AM, J6 Conn_01x05, Q1 TEMT6000X01, Q2 BC817, Q3 BC817, SW1 1101NE, SW2 1101NE, U1 MCP73871, U2 LM1117MPX-3.3_NOPB, U3 ESP32-C3-WROOM-02-H4, U4 CP2102N-A02-GQFN20, U5 USBLC6-2SC6, U6 W25Q32JVSSIQ, U7 BME280, U8 MAX4466EXK+T

Commit message: Ekspander 100x - LEDs
Connections:
- SW1 pad 2: /ESP32-C3-02/BOOT -> GND
- SW1 pad 3: GND -> /ESP32-C3-02/BOOT
- SW2 pad 2: /ESP32-C3-02/EN -> GND
- SW2 pad 3: GND -> /ESP32-C3-02/EN
